Commit message: Serve mesh files

File: urdf/07-physics.urdf (robot description, URDF)
Before this commit: robot physics, 16 links, 15 joints
Links:
- link left_gripper: geometry collision mesh filename=../12345/l_finger.dae; visual mesh filename=../12345/l_finger.dae
- link left_tip: geometry collision mesh filename=../12345/l_finger_tip.dae; visual mesh filename=../12345/l_finger_tip.dae
- link right_gripper: geometry collision mesh filename=../12345/l_finger.dae; visual mesh filename=../12345/l_finger.dae
- link right_tip: geometry collision mesh filename=../12345/l_finger_tip.dae; visual mesh filename=../12345/l_finger_tip.dae
