Commit message: Test URDF file with rvizweb renderable mesh part

File: urdf/05-visual.urdf (robot description, URDF)
Before this commit: robot visual, 16 links, 15 joints
Links:
- link left_gripper: geometry visual mesh filename=../12345/l_finger.dae
- link left_tip: geometry visual mesh filename=../12345/l_finger_tip.dae
- link right_gripper: geometry visual mesh filename=../12345/l_finger.dae
- link right_tip: geometry visual mesh filename=../12345/l_finger_tip.dae

File: urdf/06-flexible.urdf (robot description, URDF)
Before this commit: robot visual, 16 links, 15 joints
Links:
- link left_gripper: geometry visual mesh filename=../12345/l_finger.dae
- link left_tip: geometry visual mesh filename=../12345/l_finger_tip.dae
- link right_gripper: geometry visual mesh filename=../12345/l_finger.dae
- link right_tip: geometry visual mesh filename=../12345/l_finger_tip.dae
