Commit message: Update 12-PatrickB.urdf
U10 robot Base

File: urdf/12-PatrickB.urdf (robot description, URDF)
Before this commit: robot origins, 2 links, 1 joints
Links:
- removed link right_leg
- added link U10_Base; visual mesh filename=../12345/Base.stl
Joints:
- joint base_to_right_leg: child right_leg -> U10_Base; origin xyz=0 -0.22 0.25 -> xyz=0 1 0

Commit message: Update 12-PatrickB.urdf

File: urdf/12-PatrickB.urdf (robot description, URDF)
Before this commit: robot origins, 2 links, 1 joints
Links:
- added link First_Gelenk; visual mesh filename=../12345/Base.stl
Joints:
- added joint first_joint: type fixed, parent U10_Base, child First_Gelenk, origin xyz=0 1 0.5

Commit message: Update 12-PatrickB.urdf
first_joint

File: urdf/12-PatrickB.urdf (robot description, URDF)
Before this commit: robot origins, 3 links, 2 joints
Links:
- link First_Gelenk: geometry visual mesh filename=../12345/UR10_Size4_Joint_meter.stl

Commit message: Update 12-PatrickB.urdf
richtiger joint

File: urdf/12-PatrickB.urdf (robot description, URDF)
Before this commit: robot origins, 3 links, 2 joints
Joints:
- joint first_joint: origin xyz=0 1 0.5 -> xyz=0 0 0.1

Commit message: Update 12-PatrickB.urdf
test

File: urdf/12-PatrickB.urdf (robot description, URDF)
Before this commit: robot origins, 3 links, 2 joints
Links:
- added link Second_Gelenk; visual mesh filename=../12345/UR10_Size4_Joint_meter.stl
Joints:
- added joint second_joint: type continuous, parent U10_Base, child Second_Gelenk, origin xyz=0 0.086 0.090, axis 0 1 0
- joint first_joint: axis (none) -> 0 0 1; origin xyz=0 0 0.1 -> xyz=0 0 0.128; type fixed -> continuous

Commit message: Update 12-PatrickB.urdf
test

File: urdf/12-PatrickB.urdf (robot description, URDF)
Before this commit: robot origins, 4 links, 3 joints
Joints:
- joint second_joint: origin xyz=0 0.086 0.090 -> xyz=0 1 1

Commit message: Update 12-PatrickB.urdf
second gelenk

File: urdf/12-PatrickB.urdf (robot description, URDF)
Before this commit: robot origins, 4 links, 3 joints
Joints:
- joint second_joint: origin xyz=0 1 1 -> xyz=0 -0.176 0 rpy=1.571 0 0; parent U10_Base -> First_Gelenk

Commit message: Update 12-PatrickB.urdf
added upper arm link

File: urdf/12-PatrickB.urdf (robot description, URDF)
Before this commit: robot origins, 4 links, 3 joints
Links:
- added link Upper_arm; visual mesh filename=../12345/UR10_Upper_arm_meter.stl

Commit message: Update 12-PatrickB.urdf
joint origin adapted

File: urdf/12-PatrickB.urdf (robot description, URDF)
Before this commit: robot origins, 5 links, 4 joints
Joints:
- joint third_joint: origin xyz=0 0 2 rpy=0 0 0 -> xyz=0 -0.086 0 rpy=1.571 0 0

Commit message: Update 12-PatrickB.urdf
included 4thjoint

File: urdf/12-PatrickB.urdf (robot description, URDF)
Before this commit: robot origins, 5 links, 4 joints
Links:
- added link Third_Gelenk; visual mesh filename=../12345/UR10_Size3_Joint_meter.stl
Joints:
- added joint fourth_joint: type continuous, parent Second_Gelenk, child Upper_arm, origin xyz=0 0.5 0 rpy=0 0 0, axis 0 1 0

Commit message: Update 12-PatrickB.urdf
fourth joint

File: urdf/12-PatrickB.urdf (robot description, URDF)
Before this commit: robot origins, 6 links, 5 joints
Links:
- removed link Third_Gelenk
- added link Fourth_Gelenk; visual mesh filename=../12345/UR10_Size3_Joint_meter.stl
Joints:
- joint fourth_joint: child Upper_arm -> Fourth_Gelenk; parent Second_Gelenk -> Upper_arm

Commit message: Update 12-PatrickB.urdf

File: urdf/12-PatrickB.urdf (robot description, URDF)
Before this commit: robot origins, 6 links, 5 joints
Links:
- link Fourth_Gelenk: geometry visual mesh filename=../12345/UR10_Size3Joint_meter.stl
Joints:
- joint fourth_joint: origin xyz=0 0.5 0 rpy=0 0 0 -> xyz=0 0.46 0 rpy=0 0 0

Commit message: Update 12-PatrickB.urdf
test

File: urdf/12-PatrickB.urdf (robot description, URDF)
Before this commit: robot origins, 6 links, 5 joints
Joints:
- joint fourth_joint: origin xyz=0 0.46 0 rpy=0 0 0 -> xyz=0 0 0.46 rpy=0 0 0
- joint third_joint: axis 0 1 0 -> (none); origin xyz=0 -0.086 0 rpy=1.571 0 0 -> xyz=0 0 0 rpy=0 0 0; type continuous -> fixed

Commit message: Update 12-PatrickB.urdf
switched to ArmGroups

File: urdf/12-PatrickB.urdf (robot description, URDF)
Before this commit: robot origins, 6 links, 5 joints
Links:
- removed link Second_Gelenk
- added link UpperArmGroup; visual mesh filename=../12345/UR10_Size4_Joint_meter.stl
Joints:
- joint second_joint: child Second_Gelenk -> UpperArmGroup
- joint third_joint: axis (none) -> 0 1 0; parent Second_Gelenk -> UpperArmGroup; type fixed -> continuous

Commit message: Update 12-PatrickB.urdf
upperarmgroup_meter

File: urdf/12-PatrickB.urdf (robot description, URDF)
Before this commit: robot origins, 6 links, 5 joints
Links:
- link UpperArmGroup: geometry visual mesh filename=../12345/UR10_UpperArmGroup_meter.stl

Commit message: Update 12-PatrickB.urdf
lowerArmgroup

File: urdf/12-PatrickB.urdf (robot description, URDF)
Before this commit: robot origins, 6 links, 5 joints
Links:
- removed link Upper_arm
- added link LowerArmGroup; visual mesh filename=../12345/UR10_LowerArmGroup_meter.stl
Joints:
- joint fourth_joint: parent Upper_arm -> LowerArmGroup
- joint third_joint: child Upper_arm -> LowerArmGroup

Commit message: Update 12-PatrickB.urdf
joint upperarm lowerarm

File: urdf/12-PatrickB.urdf (robot description, URDF)
Before this commit: robot origins, 6 links, 5 joints
Joints:
- joint third_joint: origin xyz=0 0.1 0.61290 rpy=0 0 0 -> xyz=0 -0.02189  0.61290 rpy=0 0 -1.5708

Commit message: Update 12-PatrickB.urdf

File: urdf/12-PatrickB.urdf (robot description, URDF)
Before this commit: robot origins, 6 links, 5 joints
Links:
- link Fourth_Gelenk: geometry visual mesh filename=../12345/UR10_Size2Joint_meter.stl
Joints:
- joint fourth_joint: origin xyz=0 0 0.46 rpy=0 0 0 -> xyz=0.1 0 0.571 rpy=0 0 0

Commit message: Update 12-PatrickB.urdf

File: urdf/12-PatrickB.urdf (robot description, URDF)
Before this commit: robot origins, 6 links, 5 joints
Joints:
- joint fourth_joint: origin xyz=0.1 0 0.571 rpy=0 0 0 -> xyz=0.1 0 0.571 rpy=0 0 -1.5708

Commit message: Update 12-PatrickB.urdf
fifth_joint

File: urdf/12-PatrickB.urdf (robot description, URDF)
Before this commit: robot origins, 6 links, 5 joints
Links:
- added link Fith_Gelenk; visual mesh filename=../12345/UR10_Size2Joint_meter.stl
Joints:
- added joint fifth_joint: type continuous, parent Fourth_Gelenk, child Fith_Gelenk, origin xyz=0 0 -0.0617 rpy=0 -3.14592 -3.14592, axis 0 1 0
- joint fourth_joint: origin xyz=0.1 0 0.571 rpy=0 0 -1.5708 -> xyz=0.05601 0 0.5716 rpy=0 -3.14592 -1.5708

Commit message: Update 12-PatrickB.urdf
toolflange added

File: urdf/12-PatrickB.urdf (robot description, URDF)
Before this commit: robot origins, 7 links, 6 joints
Links:
- added link ToolFlange; visual mesh filename=../12345/UR10_ToolFlange_meter.stl
Joints:
- added joint six_joint: type continuous, parent Fith_Gelenk, child Fith_Gelenk, origin xyz=0 0 0.1 rpy=0 0 0, axis 0 1 0

Commit message: Update 12-PatrickB.urdf
six flange

File: urdf/12-PatrickB.urdf (robot description, URDF)
Before this commit: robot origins, 8 links, 7 joints
Joints:
- joint six_joint: child Fith_Gelenk -> ToolFlange; origin xyz=0 0 0.1 rpy=0 0 0 -> xyz=0 0 -0.1 rpy=0 0 0

Commit message: Update 12-PatrickB.urdf

File: urdf/12-PatrickB.urdf (robot description, URDF)
Before this commit: robot origins, 8 links, 7 joints
Joints:
- joint six_joint: origin xyz=0 0 -0.1 rpy=0 0 0 -> xyz=0 -0.054 0.0617 rpy=0 0 0

Commit message: Update 12-PatrickB.urdf
added bench

File: urdf/12-PatrickB.urdf (robot description, URDF)
Before this commit: robot origins, 8 links, 7 joints
Links:
- added link UR10_Workbench; visual mesh filename=../12345/UR10_Tisch.stl
Joints:
- added joint BenchToBase: type fixed, parent base_link, child UR10_Workbench, origin xyz=1 1 0

Commit message: Update 12-PatrickB.urdf
switched to Tisch

File: urdf/12-PatrickB.urdf (robot description, URDF)
Before this commit: robot origins, 9 links, 8 joints
Links:
- link UR10_Workbench: geometry visual mesh filename=../12345/UR10/UR10_Tisch.stl

Commit message: Update 12-PatrickB.urdf

File: urdf/12-PatrickB.urdf (robot description, URDF)
Before this commit: robot origins, 9 links, 8 joints
Links:
- link U10_Base: geometry visual mesh filename=../12345/UR10/UR10_Base.stl
- link UR10_Workbench: geometry visual mesh filename=../12345/UR10/UR10_WorkBench.stl

Commit message: Update 12-PatrickB.urdf

File: urdf/12-PatrickB.urdf (robot description, URDF)
Before this commit: robot origins, 9 links, 8 joints
Links:
- link ToolFlange: geometry visual mesh filename=../12345/UR10/UR10_ToolFlange_meter.stl
- link UpperArmGroup: geometry visual mesh filename=../12345/UR10/UR10_UpperArmGroup_meter.stl

Commit message: Update 12-PatrickB.urdf

File: urdf/12-PatrickB.urdf (robot description, URDF)
Before this commit: robot origins, 9 links, 8 joints
Links:
- link First_Gelenk: geometry visual mesh filename=../12345/UR10/UR10_Size4_Joint_meter.stl

Commit message: Update 12-PatrickB.urdf

File: urdf/12-PatrickB.urdf (robot description, URDF)
Before this commit: robot origins, 9 links, 8 joints
Links:
- added link TestUR3; visual mesh filename=../12345/UR3/shoulder.dae

Commit message: Update 12-PatrickB.urdf

File: urdf/12-PatrickB.urdf (robot description, URDF)
Before this commit: robot origins, 10 links, 8 joints
Links:
- removed link TestUR3
