Commit message: Update 13-PatrickC.urdf

File: urdf/13-PatrickC.urdf (robot description, URDF)
Before this commit: robot ur3_robot, 11 links, 10 joints
Links:
- link forearm_link: geometry collision mesh filename=package://ur_description/meshes/ur3/collision/forearm.stl; visual mesh filename=../12345/UR3/forearm.dae
- link shoulder_link: geometry collision mesh filename=package://ur_description/meshes/ur3/collision/shoulder.stl; visual mesh filename=../12345/UR3/shoulder.dae
- link upper_arm_link: geometry collision mesh filename=package://ur_description/meshes/ur3/collision/upperarm.stl; visual mesh filename=../12345/UR3/upperarm.dae
- link wrist_1_link: geometry collision mesh filename=package://ur_description/meshes/ur3/collision/wrist1.stl; visual mesh filename=../12345/UR3/wrist1.dae
- link wrist_2_link: geometry collision mesh filename=package://ur_description/meshes/ur3/collision/wrist2.stl; visual mesh filename=../12345/UR3/wrist2.dae
- link wrist_3_link: geometry collision mesh filename=package://ur_description/meshes/ur3/collision/wrist3.stl; visual mesh filename=../12345/UR3/wrist3.dae
Joints:
- joint shoulder_lift_joint: origin xyz=0 0 0 rpy=1.570796327 0 0 -> xyz=0 0 0 rpy=1.570796327 1.570796327 0
