Commit message: Update 14-PatrickD.urdf

File: urdf/14-PatrickD.urdf (robot description, URDF)
Before this commit: robot ur34_robot, 11 links, 10 joints
Links:
- removed link base_link_inertia
- removed link forearm_link
- removed link shoulder_link
- removed link upper_arm_link
- removed link wrist_1_link
- removed link wrist_2_link
- removed link wrist_3_link
- added link link_1; collision mesh filename=package://fanuc_cr35ia_support/meshes/cr35ia/collision/link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; visual mesh filename=../12345/CR35ia/link_1.stl
- added link link_2; collision mesh filename=package://fanuc_cr35ia_support/meshes/cr35ia/collision/link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; visual mesh filename=../12345/CR35ia/link_2.stl
- added link link_3; collision mesh filename=package://fanuc_cr35ia_support/meshes/cr35ia/collision/link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; visual mesh filename=../12345/CR35ia/link_3.stl
- added link link_4; collision mesh filename=package://fanuc_cr35ia_support/meshes/cr35ia/collision/link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; visual mesh filename=../12345/CR35ia/link_4.stl
- added link link_5; collision mesh filename=package://fanuc_cr35ia_support/meshes/cr35ia/collision/link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; visual mesh filename=../12345/CR35ia/link_5.stl
- added link link_6; collision mesh filename=package://fanuc_cr35ia_support/meshes/cr35ia/collision/link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; visual mesh filename=../12345/CR35ia/link_6.stl
- link base_link: geometry collision mesh filename=package://fanuc_cr35ia_support/meshes/cr35ia/collision/base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; visual mesh filename=package://fanuc_cr35ia_support/meshes/cr35ia/visual/base_li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
Joints:
- removed joint base_link-base_fixed_joint
- removed joint base_link-base_link_inertia
- removed joint elbow_joint
- removed joint flange-tool0
- removed joint shoulder_lift_joint
- removed joint shoulder_pan_joint
- removed joint wrist_1_joint
- removed joint wrist_2_joint
- removed joint wrist_3-flange
- removed joint wrist_3_joint
- added joint base_link-base: type fixed, parent base_link, child base, origin xyz=0 0 1.180 rpy=0 0 0
- added joint joint_1: type revolute, parent base_link, child link_1, origin xyz=0 0 1.180 rpy=0 0 0, axis 0 0 1, limit lower=-2.9670 upper=2.9670 effort=0 velocity=3.1415
- added joint joint_2: type revolute, parent link_1, child link_2, origin xyz=0.150 0 0 rpy=0 0 0, axis 0 1 0, limit lower=-0.7853 upper=2.0943 effort=0 velocity=3.1415
- added joint joint_3: type revolute, parent link_2, child link_3, origin xyz=0 0 0.790 rpy=0 0 0, axis 0 -1 0, limit lower=-2.1450 upper=2.3561 effort=0 velocity=3.4906
- added joint joint_4: type revolute, parent link_3, child link_4, origin xyz=0 0 0.150 rpy=0 0 0, axis -1 0 0, limit lower=-3.4906 upper=3.4906 effort=0 velocity=6.1086
- added joint joint_5: type revolute, parent link_4, child link_5, origin xyz=0.860 0 0 rpy=0 0 0, axis 0 -1 0, limit lower=-1.9198 upper=1.9198 effort=0 velocity=6.1086
- added joint joint_6: type revolute, parent link_5, child link_6, origin xyz=0.100 0 0 rpy=0 0 0, axis -1 0 0, limit lower=-7.8539 upper=7.8539 effort=0 velocity=6.9813
- added joint joint_6-flange: type fixed, parent link_6, child flange, origin xyz=0 0 0 rpy=0 0 0
- added joint link_6-tool0: type fixed, parent flange, child tool0, origin xyz=0 0 0 rpy=3.141592653589793 -1.5707963267948966 0

Commit message: Update 14-PatrickD.urdf

File: urdf/14-PatrickD.urdf (robot description, URDF)
Before this commit: robot fanuc_cr35ia, 10 links, 9 joints
Links:
- link base_link: geometry collision mesh filename=package://fanuc_cr35ia_support/meshes/cr35ia/collision/base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; visual mesh filename=../12345/CR35ia/base_link.stl
