Commit message: Update 11-PatrickA.urdf
added more code

File: urdf/11-PatrickA.urdf (robot description, URDF)
Before this commit: robot GoldbarrenGroup, 2 links, 1 joints
Links:
- link right_leg: geometry visual mesh filename=package://GoldbarrenGroup_description/meshes/GoldbarrenPart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 scale=0.03

Commit message: Update 11-PatrickA.urdf
changed for webserver path in geometry

File: urdf/11-PatrickA.urdf (robot description, URDF)
Before this commit: robot GoldbarrenGroup, 2 links, 1 joints
Links:
- link right_leg: geometry visual mesh filename=../12345/GoldbarrenPart1.stl

Commit message: Update 11-PatrickA.urdf
test with dae

File: urdf/11-PatrickA.urdf (robot description, URDF)
Before this commit: robot GoldbarrenGroup, 2 links, 1 joints
Links:
- link right_leg: geometry visual mesh filename=../12345/l_finger_tip.dae

Commit message: Update 11-PatrickA.urdf
test again

File: urdf/11-PatrickA.urdf (robot description, URDF)
Before this commit: robot GoldbarrenGroup, 2 links, 1 joints
Links:
- link right_leg: geometry visual mesh filename=../12345/base.stl

Commit message: Update 11-PatrickA.urdf
added 2nd goldbarren

File: urdf/11-PatrickA.urdf (robot description, URDF)
Before this commit: robot GoldbarrenGroup, 2 links, 1 joints
Links:
- added link GoldbarrenPart1:2, mass 12.0785; visual mesh filename=../12345/GoldbarrenPart1.stl
Joints:
- added joint Starr:1: type fixed, parent , child , origin xyz= rpy=0   0   0

Commit message: Update 11-PatrickA.urdf
role back

File: urdf/11-PatrickA.urdf (robot description, URDF)
Before this commit: robot GoldbarrenGroup, 3 links, 2 joints
Links:
- removed link GoldbarrenPart1:2
Joints:
- removed joint Starr:1

Commit message: Update 11-PatrickA.urdf
visual got the inventor-name"GoldbarrenPart1:1"

File: urdf/11-PatrickA.urdf (robot description, URDF)
Before this commit: robot GoldbarrenGroup, 2 links, 1 joints
Links:
- removed link right_leg
- added link GoldbarrenPart1:1; visual mesh filename=../12345/GoldbarrenPart1.stl
Joints:
- joint base_to_right_leg: child right_leg -> GoldbarrenPart1:1

Commit message: Update 11-PatrickA.urdf
added scale

File: urdf/11-PatrickA.urdf (robot description, URDF)
Before this commit: robot GoldbarrenGroup, 2 links, 1 joints
Links:
- link GoldbarrenPart1:1: geometry visual mesh filename=../12345/GoldbarrenPart1.stl scale=0.5

Commit message: Update 11-PatrickA.urdf
with second joint but without scale

File: urdf/11-PatrickA.urdf (robot description, URDF)
Before this commit: robot GoldbarrenGroup, 2 links, 1 joints
Links:
- added link GoldbarrenPart1:2; visual mesh filename=../12345/GoldbarrenPart1.stl
- link GoldbarrenPart1:1: geometry visual mesh filename=../12345/GoldbarrenPart1.stl
Joints:
- added joint starr: type fixed, parent GoldbarrenPart1:1, child GoldbarrenPart1:2, origin xyz=0 0 0

Commit message: Update 11-PatrickA.urdf
changed origin

File: urdf/11-PatrickA.urdf (robot description, URDF)
Before this commit: robot GoldbarrenGroup, 3 links, 2 joints
Joints:
- joint starr: origin xyz=0 0 0 -> xyz=0 200 0

Commit message: Update 11-PatrickA.urdf
adapted jonit

File: urdf/11-PatrickA.urdf (robot description, URDF)
Before this commit: robot GoldbarrenGroup, 3 links, 2 joints
Joints:
- removed joint starr
- added joint Starr:1: type fixed, parent GoldbarrenPart1:1, child GoldbarrenPart1:2, origin xyz=0 200 0 rpy=0 0 0

Commit message: Update 11-PatrickA.urdf
check units via zylinder

File: urdf/11-PatrickA.urdf (robot description, URDF)
Before this commit: robot GoldbarrenGroup, 3 links, 2 joints
Links:
- link base_link: geometry visual cylinder length=1 radius=0.2
Joints:
- joint base_to_right_leg: origin xyz=0 -0.22 0.25 -> xyz=50 0 0.25

Commit message: Update 11-PatrickA.urdf
unit test with zylinder length

File: urdf/11-PatrickA.urdf (robot description, URDF)
Before this commit: robot GoldbarrenGroup, 3 links, 2 joints
Links:
- link base_link: geometry visual cylinder length=42 radius=0.2

Commit message: Update 11-PatrickA.urdf
asci stl

File: urdf/11-PatrickA.urdf (robot description, URDF)
Before this commit: robot GoldbarrenGroup, 3 links, 2 joints
Links:
- link GoldbarrenPart1:2: geometry visual mesh filename=../12345/GoldbarrenPart1_Ascii.stl

Commit message: Update 11-PatrickA.urdf
Tried with size adaptoin

File: urdf/11-PatrickA.urdf (robot description, URDF)
Before this commit: robot GoldbarrenGroup, 3 links, 2 joints
Links:
- link GoldbarrenPart1:2: geometry visual mesh filename=../12345/GoldbarrenPart1_AsciiMeter.stl

Commit message: Update 11-PatrickA.urdf
both ascii meter

File: urdf/11-PatrickA.urdf (robot description, URDF)
Before this commit: robot GoldbarrenGroup, 3 links, 2 joints
Links:
- link GoldbarrenPart1:1: geometry visual mesh filename=../12345/GoldbarrenPart1_AsciiMeter.stl

Commit message: Update 11-PatrickA.urdf
cm

File: urdf/11-PatrickA.urdf (robot description, URDF)
Before this commit: robot GoldbarrenGroup, 3 links, 2 joints
Links:
- link GoldbarrenPart1:1: geometry visual mesh filename=../12345/GoldbarrenPart1_cm.stl
- link GoldbarrenPart1:2: geometry visual mesh filename=../12345/GoldbarrenPart1_cm.stl

Commit message: Update 11-PatrickA.urdf
reduced distances

File: urdf/11-PatrickA.urdf (robot description, URDF)
Before this commit: robot GoldbarrenGroup, 3 links, 2 joints
Joints:
- joint Starr:1: origin xyz=0 200 0 rpy=0 0 0 -> xyz=0 20 0 rpy=0 0 0

Commit message: Update 11-PatrickA.urdf

File: urdf/11-PatrickA.urdf (robot description, URDF)
Before this commit: robot GoldbarrenGroup, 3 links, 2 joints
Links:
- link GoldbarrenPart1:2: geometry visual mesh filename=../12345/GoldbarrenPart1_meter.stl

Commit message: Update 11-PatrickA.urdf
changed to values ...

File: urdf/11-PatrickA.urdf (robot description, URDF)
Before this commit: robot GoldbarrenGroup, 3 links, 2 joints
Joints:
- joint Starr:1: origin xyz=0 20 0 rpy=0 0 0 -> xyz=0 0 0 rpy=0 0 0
- joint base_to_right_leg: origin xyz=50 0 0.25 -> xyz=30 0 0.25

Commit message: Update 11-PatrickA.urdf

File: urdf/11-PatrickA.urdf (robot description, URDF)
Before this commit: robot GoldbarrenGroup, 3 links, 2 joints
Joints:
- joint base_to_right_leg: origin xyz=30 0 0.25 -> xyz=3 0 0.25

Commit message: Update 11-PatrickA.urdf
changed name of visual

File: urdf/11-PatrickA.urdf (robot description, URDF)
Before this commit: robot GoldbarrenGroup, 3 links, 2 joints
Links:
- removed link GoldbarrenPart1:2
- added link Stehtisch_meter:1; visual mesh filename=../12345/Stehtisch_meter.stl
Joints:
- joint Starr:1: child GoldbarrenPart1:2 -> Stehtisch_meter:1

Commit message: Update 11-PatrickA.urdf
included schutzzaun

File: urdf/11-PatrickA.urdf (robot description, URDF)
Before this commit: robot GoldbarrenGroup, 3 links, 2 joints
Links:
- added link schutzzaun_meter; visual mesh filename=../12345/schutzzaun_meter.stl
Joints:
- joint Starr:1: child Stehtisch_meter:1 -> schutzzaun_meter

Commit message: Update 11-PatrickA.urdf
zaun verschoben

File: urdf/11-PatrickA.urdf (robot description, URDF)
Before this commit: robot GoldbarrenGroup, 4 links, 2 joints
Joints:
- joint Starr:1: origin xyz=0 0 0 rpy=0 0 0 -> xyz=0 5 0 rpy=0 0 0

Commit message: Update 11-PatrickA.urdf
bauzaun auf baselink

File: urdf/11-PatrickA.urdf (robot description, URDF)
Before this commit: robot GoldbarrenGroup, 4 links, 2 joints
Joints:
- joint Starr:1: parent GoldbarrenPart1:1 -> base_link

Commit message: Update 11-PatrickA.urdf
zaun verschoen

File: urdf/11-PatrickA.urdf (robot description, URDF)
Before this commit: robot GoldbarrenGroup, 4 links, 2 joints
Joints:
- joint Starr:1: child schutzzaun_meter -> Stehtisch_meter:1; origin xyz=0 5 0 rpy=0 0 0 -> xyz=0 0 0 rpy=0 0 0; parent base_link -> GoldbarrenPart1:1

Commit message: Update 11-PatrickA.urdf
test

File: urdf/11-PatrickA.urdf (robot description, URDF)
Before this commit: robot GoldbarrenGroup, 4 links, 2 joints
Joints:
- joint Starr:1: origin xyz=0 0 0 rpy=0 0 0 -> xyz=5 0 0 rpy=0 0 0
- joint base_to_right_leg: origin xyz=3 0 0.25 -> xyz=0 0 0.25

Commit message: Update 11-PatrickA.urdf

File: urdf/11-PatrickA.urdf (robot description, URDF)
Before this commit: robot GoldbarrenGroup, 4 links, 2 joints
Joints:
- joint base_to_right_leg: parent base_link -> schutzzaun_meter

Commit message: Update 11-PatrickA.urdf
test

File: urdf/11-PatrickA.urdf (robot description, URDF)
Before this commit: robot GoldbarrenGroup, 4 links, 2 joints
Joints:
- added joint Starr:2: type fixed, parent GoldbarrenPart1:1, child Stehtisch_meter:1, origin xyz=5 0 0 rpy=0 0 0
- joint Starr:1: child Stehtisch_meter:1 -> schutzzaun_meter; origin xyz=5 0 0 rpy=0 0 0 -> xyz=0 5 0.5 rpy=0 0 0; parent GoldbarrenPart1:1 -> base_link

Commit message: Update 11-PatrickA.urdf
with fanuc

File: urdf/11-PatrickA.urdf (robot description, URDF)
Before this commit: robot GoldbarrenGroup, 4 links, 3 joints
Links:
- added link fanuc; visual mesh filename=../12345/CR35Fanuc_meter.stl
- added link schutzzaun_meter2; visual mesh filename=../12345/schutzzaun_meter.stl
- added link schutzzaun_meter3; visual mesh filename=../12345/schutzzaun_meter.stl
Joints:
- added joint Starr:3: type fixed, parent base_link, child schutzzaun_meter3, origin xyz=-2 4 0.2 rpy=0 0 0
- added joint Starr:4: type fixed, parent base_link, child Stehtisch_meter:1, origin xyz=-2 2 0 rpy=0 0 0
- joint Starr:1: origin xyz=0 5 0.5 rpy=0 0 0 -> xyz=0 4 0.2 rpy=0 0 0
- joint Starr:2: child Stehtisch_meter:1 -> schutzzaun_meter2; origin xyz=5 0 0 rpy=0 0 0 -> xyz=2 4 0.2 rpy=0 0 -0.8; parent GoldbarrenPart1:1 -> base_link
- joint base_to_right_leg: origin xyz=0 0 0.25 -> xyz=0 0 0.8; parent schutzzaun_meter -> Stehtisch_meter:1

Commit message: Update 11-PatrickA.urdf
with robot

File: urdf/11-PatrickA.urdf (robot description, URDF)
Before this commit: robot GoldbarrenGroup, 7 links, 5 joints
Joints:
- added joint Starr:5: type fixed, parent base_link, child fanuc, origin xyz=-2 2 0 rpy=0 0 0
- joint Starr:4: origin xyz=-2 2 0 rpy=0 0 0 -> xyz=2 2 0 rpy=0 0 0
- joint base_to_right_leg: origin xyz=0 0 0.8 -> xyz=0.1 0.3 1.05

Commit message: Update 11-PatrickA.urdf

File: urdf/11-PatrickA.urdf (robot description, URDF)
Before this commit: robot GoldbarrenGroup, 7 links, 6 joints
Links:
- link schutzzaun_meter: geometry visual mesh filename=../12345/Fences/SafetyFence_2000x2100.stl
- link schutzzaun_meter2: geometry visual mesh filename=../12345/Fences/SafetyFence_2000x2100.stl
- link schutzzaun_meter3: geometry visual mesh filename=../12345/Fences/SafetyFence_2000x2100.stl

Commit message: Update 11-PatrickA.urdf

File: urdf/11-PatrickA.urdf (robot description, URDF)
Before this commit: robot GoldbarrenGroup, 7 links, 6 joints
Links:
- link fanuc: geometry visual mesh filename=../12345/CR35ia/CR35ia_StaticDummy.stl
