Commit message: Update ur5.urdf

File: meshes/UR5/ur5.urdf (robot description, URDF)
Before this commit: robot ur5, 11 links, 10 joints
Links:
- link base_link: geometry collision mesh filename=package://ur_description/meshes/ur5/collision/base.stl; visual mesh filename=../12345/UR5/base.dae
- link forearm_link: geometry collision mesh filename=package://ur_description/meshes/ur5/collision/forearm.stl; visual mesh filename=../12345/UR5/forearm.dae
- link shoulder_link: geometry collision mesh filename=package://ur_description/meshes/ur5/collision/shoulder.stl; visual mesh filename=../12345/UR5/shoulder.dae
- link upper_arm_link: geometry collision mesh filename=package://ur_description/meshes/ur5/collision/upperarm.stl; visual mesh filename=../12345/UR5/upperarm.dae
- link wrist_1_link: geometry collision mesh filename=package://ur_description/meshes/ur5/collision/wrist1.stl; visual mesh filename=../12345/UR5/wrist1.dae
- link wrist_2_link: geometry collision mesh filename=package://ur_description/meshes/ur5/collision/wrist2.stl; visual mesh filename=../12345/UR5/wrist2.dae
- link wrist_3_link: geometry collision mesh filename=package://ur_description/meshes/ur5/collision/wrist3.stl; visual mesh filename=../12345/UR5/wrist3.dae
