Commit message: Update ur10.urdf

File: meshes/UR10/ur10.urdf (robot description, URDF)
Before this commit: robot ur10_robot, 11 links, 10 joints
Links:
- link base_link_inertia: geometry collision mesh filename=package://ur_description/meshes/ur10/collision/base.stl; visual mesh filename=../12345/UR10/base.dae
- link forearm_link: geometry collision mesh filename=package://ur_description/meshes/ur10/collision/forearm.stl; visual mesh filename=../12345/UR10/forearm.dae
- link shoulder_link: geometry collision mesh filename=package://ur_description/meshes/ur10/collision/shoulder.stl; visual mesh filename=../12345/UR10/shoulder.dae
- link upper_arm_link: geometry collision mesh filename=package://ur_description/meshes/ur10/collision/upperarm.stl; visual mesh filename=../12345/UR10/upperarm.dae
- link wrist_1_link: geometry collision mesh filename=package://ur_description/meshes/ur10/collision/wrist1.stl; visual mesh filename=../12345/UR10/wrist1.dae
- link wrist_2_link: geometry collision mesh filename=package://ur_description/meshes/ur10/collision/wrist2.stl; visual mesh filename=../12345/UR10/wrist2.dae
- link wrist_3_link: geometry collision mesh filename=package://ur_description/meshes/ur10/collision/wrist3.stl; visual mesh filename=../12345/UR10/wrist3.dae

Commit message: Update ur10.urdf

File: meshes/UR10/ur10.urdf (robot description, URDF)
Before this commit: robot ur10_robot, 11 links, 10 joints
Joints:
- joint shoulder_lift_joint: origin xyz=0 0 0 rpy=1.570796327 0 0 -> xyz=0 0 0 rpy=1.570796327 1.570796327 0
