Commit message: Update Scenario_Bv02.urdf

File: urdf/Scenario_B/Scenario_Bv02.urdf (robot description, URDF)
Before this commit: robot ur10_robot, 13 links, 12 joints
Links:
- added link Plate_Bench; visual mesh filename=../12345/Workstations/Slottted_Plate_Bench_700x1500.stl
Joints:
- joint BenchToScenario: child UR10_Workbench -> Plate_Bench; origin xyz=0 2 0.9 -> xyz=0 -2 0.9

Commit message: Update Scenario_Bv02.urdf

File: urdf/Scenario_B/Scenario_Bv02.urdf (robot description, URDF)
Before this commit: robot ur10_robot, 14 links, 12 joints
Links:
- link base_link: geometry visual cylinder length=22 radius=0.1
Joints:
- added joint BenchTobaseLink: type fixed, parent base_link, child UR10_Workbench, origin xyz=0 4 0.9
- joint BenchToScenario: origin xyz=0 -2 0.9 -> xyz=0 2 0.9

Commit message: Update Scenario_Bv02.urdf

File: urdf/Scenario_B/Scenario_Bv02.urdf (robot description, URDF)
Before this commit: robot ur10_robot, 14 links, 13 joints
Joints:
- joint BenchTobaseLink: origin xyz=0 4 0.9 -> xyz=-1.5 2 0.9

Commit message: Update Scenario_Bv02.urdf

File: urdf/Scenario_B/Scenario_Bv02.urdf (robot description, URDF)
Before this commit: robot ur10_robot, 14 links, 13 joints
Links:
- link Plate_Bench: geometry visual mesh filename=../12345/Workstations/Slotted_Plate_Bench_700x1500.stl
- link UR10_Workbench: geometry visual mesh filename=../12345/Workstations/Slotted_Plate_Bench_700x1500.stl
