Commit message: Update Scenario_Bv01.urdf

File: urdf/Scenario_B/Scenario_Bv01.urdf (robot description, URDF)
Before this commit: robot ur10_robot, 11 links, 10 joints
Links:
- added link UR10_Workbench; visual mesh filename=../12345/meshes/Workstations/Slottted_Plate_Bench_700x1500.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
Joints:
- added joint BenchToBase: type fixed, parent base_link, child UR10_Workbench, origin xyz=0 2 0.9

Commit message: Update Scenario_Bv01.urdf

File: urdf/Scenario_B/Scenario_Bv01.urdf (robot description, URDF)
Before this commit: robot ur10_robot, 13 links, 12 joints
Links:
- link UR10_Workbench: geometry visual mesh filename=../12345/Workstations/Slotted_Plate_Bench_700x1500.stl

Commit message: Update Scenario_Bv01.urdf

File: urdf/Scenario_B/Scenario_Bv01.urdf (robot description, URDF)
Before this commit: robot ur10_robot, 13 links, 12 joints
Links:
- link Scenario_base: geometry visual cylinder length=1 radius=0.02
