Commit message: Update Fences.urdf

File: meshes/Fences/Fences.urdf (robot description, URDF)
Before this commit: robot Workstations, 3 links, 2 joints
Links:
- added link PartitionWall_2100x790; visual mesh filename=../12345/Fences/PartitionWall_2100x790.stl
Joints:
- removed joint PartitionWallTobaseLink
- added joint PartitionWall1800TobaseLink: type fixed, parent base_link, child PartitionWall_1800x790, origin xyz=0 2 0
- added joint PartitionWall2100TobaseLink: type fixed, parent base_link, child PartitionWall_2100x790, origin xyz=-2 2 0

Commit message: Update Fences.urdf

File: meshes/Fences/Fences.urdf (robot description, URDF)
Before this commit: robot Workstations, 4 links, 3 joints
Links:
- link base_link: geometry visual cylinder length=1 radius=0.02
