Commit message: Update 05-visual.urdf

File: urdf/00_BasicSamples/05-visual.urdf (robot description, URDF)
Before this commit: robot visual, 16 links, 15 joints
Links:
- link left_gripper: geometry visual mesh filename=../12345/00_BasicSamples/l_finger.dae
- link left_tip: geometry visual mesh filename=../12345/00_BasicSamples/l_finger_tip.dae
- link right_gripper: geometry visual mesh filename=../12345/00_BasicSamples/l_finger.dae
- link right_tip: geometry visual mesh filename=../12345/00_BasicSamples/l_finger_tip.dae
