Commit message: Update 10-osaca2.urdf

File: urdf/00_BasicSamples/10-osaca2.urdf (robot description, URDF)
Before this commit: robot osaca2, 6 links, 5 joints
Links:
- link a1_link: geometry visual mesh filename=../12345/00_BasicSamples/a1.stl
- link a2_link: geometry visual mesh filename=../12345/00_BasicSamples/a2.stl
- link a3_link: geometry visual mesh filename=../12345/00_BasicSamples/a3.stl
- link base_link: geometry visual mesh filename=../12345/00_BasicSamples/base.stl

Commit message: Update 10-osaca2.urdf

File: urdf/00_BasicSamples/10-osaca2.urdf (robot description, URDF)
Before this commit: robot osaca2, 6 links, 5 joints
Links:
- link box_link: geometry visual mesh filename=../12345/00_BasicSamples/box.stl
