Commit message: Update ScenarioD_Variant01.urdf

File: urdf/Scenario_D/ScenarioD_Variant01.urdf (robot description, URDF)
Before this commit: robot fanuc_cr35ia, 10 links, 9 joints
Links:
- added link ConveyerTable; visual mesh filename=../12345/Workstations/transportband02.stl
- added link robot_base; collision mesh filename=package://fanuc_cr35ia_support/meshes/cr35ia/collision/base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; visual mesh filename=../12345/CR35ia/base_link.stl
- link base_link: geometry visual cylinder length=1 radius=0.02
Joints:
- added joint ConveyerTableTobaseLink: type fixed, parent base_link, child ConveyerTable, origin xyz=-1 1 0
- added joint RobotBaseTobaseLink: type fixed, parent base_link, child robot_base, origin xyz=1 1 0
- joint joint_1: parent base_link -> robot_base

Commit message: Update ScenarioD_Variant01.urdf

File: urdf/Scenario_D/ScenarioD_Variant01.urdf (robot description, URDF)
Before this commit: robot fanuc_cr35ia, 12 links, 11 joints
Links:
- removed link ConveyerTable
- added link ConveyerTable01; visual mesh filename=../12345/Workstations/transportband02.stl
- added link ConveyerTable02; visual mesh filename=../12345/Workstations/transportband02.stl
- added link WoodPlate_Bench_700x1500x900; visual mesh filename=../12345/Workstations/WoodPlate_Bench_700x1500x900.stl
Joints:
- removed joint ConveyerTableTobaseLink
- added joint ConveyerTable01TobaseLink: type fixed, parent base_link, child ConveyerTable01, origin xyz=1 -1.2 0.9
- added joint ConveyerTable02TobaseLink: type fixed, parent base_link, child ConveyerTable02, origin xyz=1 1.2 0.9
- added joint WoodPlate_Bench_700x1500x900TobaseLink: type fixed, parent base_link, child WoodPlate_Bench_700x1500x900, origin xyz=3 -0.75 0.9 rpy=0 0 1.571
- joint RobotBaseTobaseLink: origin xyz=1 1 0 -> xyz=1 0 0
