Commit message: Update OnrobotRG2.urdf

File: meshes/Grippers/OnrobotRG2.urdf (robot description, URDF)
Before this commit: robot onrobot_rg2_model, 7 links, 6 joints
Links:
- link left_outer_knuckle: geometry collision mesh filename=package://onrobot_rg2_visualization/meshes/collision/outer_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; visual mesh filename=../12345/Grippers/OnrobotRG2/visual/outer_knuckle.stl
