Commit message: Update OnrobotRG2.urdf

File: meshes/Grippers/OnrobotRG2/OnrobotRG2.urdf (robot description, URDF)
Before this commit: robot onrobot_rg2_model, 7 links, 6 joints
Links:
- link left_inner_finger: geometry collision mesh filename=package://onrobot_rg2_visualization/meshes/collision/inner_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; visual mesh filename=../12345/Grippers/OnrobotRG2/visual/inner_finger.stl
- link left_inner_knuckle: geometry collision mesh filename=package://onrobot_rg2_visualization/meshes/collision/inner_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; visual mesh filename=../12345/Grippers/OnrobotRG2/visual/inner_knuckle.stl
- link onrobot_rg2_base_link: geometry collision mesh filename=package://onrobot_rg2_visualization/meshes/collision/base_l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; visual mesh filename=../12345/Grippers/OnrobotRG2/visual/base_link.stl
- link right_inner_finger: geometry collision mesh filename=package://onrobot_rg2_visualization/meshes/collision/inner_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; visual mesh filename=../12345/Grippers/OnrobotRG2/visual/inner_finger.stl
- link right_inner_knuckle: geometry collision mesh filename=package://onrobot_rg2_visualization/meshes/collision/inner_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; visual mesh filename=../12345/Grippers/OnrobotRG2/visual/inner_knuckle.stl
- link right_outer_knuckle: geometry collision mesh filename=package://onrobot_rg2_visualization/meshes/collision/outer_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; visual mesh filename=../12345/Grippers/OnrobotRG2/visual/outer_knuckle.stl

Commit message: Update OnrobotRG2.urdf

File: meshes/Grippers/OnrobotRG2/OnrobotRG2.urdf (robot description, URDF)
Before this commit: robot onrobot_rg2_model, 7 links, 6 joints
Links:
- added link base_link; visual cylinder length=1 radius=0.02
Joints:
- added joint test: type fixed, parent base_link, child onrobot_rg2_base_link, origin xyz=0.3 0 0
