Commit message: Update workpieces.urdf

File: meshes/Workpieces/workpieces.urdf (robot description, URDF)
Before this commit: robot Workpieces, 2 links, 1 joints
Links:
- removed link template
- added link flower_vase_170x118; visual mesh filename=../12345/Fences/flower_vase_170x118.stl
Joints:
- joint PartitionWall1800TobaseLink: child PartitionWall_1800x790 -> flower_vase_170x118; origin xyz=0 2 0 -> xyz=1 1 0

Commit message: Update workpieces.urdf

File: meshes/Workpieces/workpieces.urdf (robot description, URDF)
Before this commit: robot Workpieces, 2 links, 1 joints
Links:
- link flower_vase_170x118: geometry visual mesh filename=../12345/Workpieces/flower_vase_170x118.stl

Commit message: Update workpieces.urdf

File: meshes/Workpieces/workpieces.urdf (robot description, URDF)
Before this commit: robot Workpieces, 2 links, 1 joints
Links:
- added link Monitor_965x710; visual mesh filename=../12345/Workpieces/Monitor_965x710.stl
Joints:
- added joint Monitor_965x710TobaseLink: type fixed, parent base_link, child Monitor_965x710, origin xyz=1 -1 0

Commit message: Update workpieces.urdf

File: meshes/Workpieces/workpieces.urdf (robot description, URDF)
Before this commit: robot Workpieces, 3 links, 2 joints
Links:
- added link flower_vase_162x185; visual mesh filename=../12345/Workpieces/flower_vase_170x118.stl
Joints:
- removed joint PartitionWall1800TobaseLink
- added joint flower_vase_162x185TobaseLink: type fixed, parent base_link, child flower_vase_170x118, origin xyz=1 1 0
- added joint flower_vase_170x118TobaseLink: type fixed, parent base_link, child flower_vase_170x118, origin xyz=1 1 0

Commit message: Update workpieces.urdf

File: meshes/Workpieces/workpieces.urdf (robot description, URDF)
Before this commit: robot Workpieces, 4 links, 3 joints
Joints:
- joint flower_vase_162x185TobaseLink: origin xyz=1 1 0 -> xyz=1 1.5 0

Commit message: Update workpieces.urdf

File: meshes/Workpieces/workpieces.urdf (robot description, URDF)
Before this commit: robot Workpieces, 4 links, 3 joints
Joints:
- joint flower_vase_162x185TobaseLink: child flower_vase_170x118 -> flower_vase_162x185

Commit message: Update workpieces.urdf

File: meshes/Workpieces/workpieces.urdf (robot description, URDF)
Before this commit: robot Workpieces, 4 links, 3 joints
Links:
- link flower_vase_162x185: geometry visual mesh filename=../12345/Workpieces/flower_vase_162x185.stl

Commit message: Update workpieces.urdf

File: meshes/Workpieces/workpieces.urdf (robot description, URDF)
Before this commit: robot Workpieces, 4 links, 3 joints
Links:
- added link FittingPipe_694x392_PN40; visual mesh filename=../12345/Workpieces/FittingPipe_694x392_PN40.stl
- added link Flange_270x68_PN40; visual mesh filename=../12345/Workpieces/Flange_270x68_PN40.stl

Commit message: Update workpieces.urdf

File: meshes/Workpieces/workpieces.urdf (robot description, URDF)
Before this commit: robot Workpieces, 6 links, 3 joints
Joints:
- added joint FittingPipe_694x392_PN40TobaseLink: type fixed, parent base_link, child FittingPipe_694x392_PN40, origin xyz=1 -1 0
- added joint Flange_270x68_PN40TobaseLink: type fixed, parent base_link, child Flange_270x68_PN40, origin xyz=1 -1 0

Commit message: Update workpieces.urdf

File: meshes/Workpieces/workpieces.urdf (robot description, URDF)
Before this commit: robot Workpieces, 6 links, 5 joints
Joints:
- joint FittingPipe_694x392_PN40TobaseLink: origin xyz=1 -1 0 -> xyz=1.5 -1 0
- joint Flange_270x68_PN40TobaseLink: origin xyz=1 -1 0 -> xyz=2 -1 0

Commit message: Update workpieces.urdf

File: meshes/Workpieces/workpieces.urdf (robot description, URDF)
Before this commit: robot Workpieces, 6 links, 5 joints
Joints:
- joint FittingPipe_694x392_PN40TobaseLink: origin xyz=1.5 -1 0 -> xyz=-1.5 -1 0
- joint Flange_270x68_PN40TobaseLink: origin xyz=2 -1 0 -> xyz=-2 -1 0

Commit message: Update workpieces.urdf

File: meshes/Workpieces/workpieces.urdf (robot description, URDF)
Before this commit: robot Workpieces, 6 links, 5 joints
Links:
- added link BallBearings_SKF6256_500x80; visual mesh filename=../12345/Workpieces/BallBearings_SKF6256_500x80.stl
Joints:
- added joint BallBearings_SKF6256_500x80TobaseLink: type fixed, parent base_link, child BallBearings_SKF6256_500x80, origin xyz=-2 -0.5 0

Commit message: Update workpieces.urdf

File: meshes/Workpieces/workpieces.urdf (robot description, URDF)
Before this commit: robot Workpieces, 7 links, 6 joints
Joints:
- joint BallBearings_SKF6256_500x80TobaseLink: origin xyz=-2 -0.5 0 -> xyz=-2 -0 0

Commit message: Update workpieces.urdf

File: meshes/Workpieces/workpieces.urdf (robot description, URDF)
Before this commit: robot Workpieces, 7 links, 6 joints
Links:
- added link BallBearings_SKF6238_146x55; visual mesh filename=../12345/Workpieces/BallBearings_SKF6238_146x55.stl
Joints:
- added joint BallBearings_SKF6238_146x55TobaseLink: type fixed, parent base_link, child BallBearings_SKF6238_146x55, origin xyz=-1 -0 0
