Commit message: Update ScenarioC_Variant01.urdf

File: urdf/Scenario_C/ScenarioC_Variant01.urdf (robot description, URDF)
Before this commit: robot ur5, 11 links, 10 joints
Links:
- added link left_inner_finger, mass 0.05; collision mesh filename=package://onrobot_rg2_visualization/meshes/collision/inner_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; visual mesh filename=../12345/Grippers/OnrobotRG2/visual/inner_finger.stl
- added link left_inner_knuckle, mass 0.05; collision mesh filename=package://onrobot_rg2_visualization/meshes/collision/inner_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; visual mesh filename=../12345/Grippers/OnrobotRG2/visual/inner_knuckle.stl
- added link left_outer_knuckle, mass 0.05; collision mesh filename=package://onrobot_rg2_visualization/meshes/collision/outer_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; visual mesh filename=../12345/Grippers/OnrobotRG2/visual/outer_knuckle.stl
- added link onrobot_rg2_base_link, mass 0.7; collision mesh filename=package://onrobot_rg2_visualization/meshes/collision/base_l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; visual mesh filename=../12345/Grippers/OnrobotRG2/visual/base_link.stl
- added link right_inner_finger, mass 0.05; collision mesh filename=package://onrobot_rg2_visualization/meshes/collision/inner_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; visual mesh filename=../12345/Grippers/OnrobotRG2/visual/inner_finger.stl
- added link right_inner_knuckle, mass 0.05; collision mesh filename=package://onrobot_rg2_visualization/meshes/collision/inner_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; visual mesh filename=../12345/Grippers/OnrobotRG2/visual/inner_knuckle.stl
- added link right_outer_knuckle, mass 0.05; collision mesh filename=package://onrobot_rg2_visualization/meshes/collision/outer_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; visual mesh filename=../12345/Grippers/OnrobotRG2/visual/outer_knuckle.stl
Joints:
- added joint finger_joint: type revolute, parent onrobot_rg2_base_link, child left_outer_knuckle, origin xyz=0 -0.017178 0.125797 rpy=0 0 0, axis -1 0 0, limit lower=-0.558505 upper=0.785398 effort=1000 velocity=2.0
- added joint left_inner_finger_joint: type revolute, parent left_outer_knuckle, child left_inner_finger, origin xyz=0 -0.039592 0.038177000000000016 rpy=0 0 0, axis 1 0 0, limit lower=-0.872665 upper=0.872665 effort=1000 velocity=2.0, mimic joint=finger_joint multiplier=1 offset=0
- added joint left_inner_knuckle_joint: type revolute, parent onrobot_rg2_base_link, child left_inner_knuckle, origin xyz=0 -0.007678 0.1422970 rpy=0 0 0.0, axis 1 0 0, limit lower=-0.558505 upper=0.785398 effort=1000 velocity=2.0, mimic joint=finger_joint multiplier=-1 offset=0
- added joint right_inner_finger_joint: type revolute, parent right_outer_knuckle, child right_inner_finger, origin xyz=0 -0.039592 0.038177000000000016 rpy=0 0 0, axis 1 0 0, limit lower=-0.872665 upper=0.872665 effort=1000 velocity=2.0, mimic joint=finger_joint multiplier=1 offset=0
- added joint right_inner_knuckle_joint: type revolute, parent onrobot_rg2_base_link, child right_inner_knuckle, origin xyz=0 0.007678 0.1422970 rpy=0 0 -3.141592653589793, axis 1 0 0, limit lower=-0.558505 upper=0.785398 effort=1000 velocity=2.0, mimic joint=finger_joint multiplier=-1 offset=0
- added joint right_outer_knuckle_joint: type revolute, parent onrobot_rg2_base_link, child right_outer_knuckle, origin xyz=0 0.017178 0.125797 rpy=0 0 3.141592653589793, axis 1 0 0, limit lower=-0.558505 upper=0.785398 effort=1000 velocity=2.0, mimic joint=finger_joint multiplier=-1 offset=0
- joint wrist_3_link-tool0_fixed_joint: child tool0 -> onrobot_rg2_base_link

Commit message: Update ScenarioC_Variant01.urdf

File: urdf/Scenario_C/ScenarioC_Variant01.urdf (robot description, URDF)
Before this commit: robot ur5, 18 links, 16 joints
Links:
- removed link tool0
Joints:
- joint shoulder_lift_joint: origin xyz=0.0 0.13585 0.0 rpy=0.0 1.5707963267948966 0.0 -> xyz=0.0 0.13585 0.0 rpy=0.0 0.0 0.0
