Commit message: Update and rename ScenarioC_Variant01.urdf to ScenarioC_Variant02.urdf

File: urdf/Scenario_C/ScenarioC_Variant02.urdf (robot description, URDF)
Before this commit: robot ur3_robot, 11 links, 10 joints
Links:
- added link left_inner_finger, mass 0.05; collision mesh filename=package://onrobot_rg2_visualization/meshes/collision/inner_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; visual mesh filename=../12345/Grippers/OnrobotRG2/visual/inner_finger.stl
- added link left_inner_knuckle, mass 0.05; collision mesh filename=package://onrobot_rg2_visualization/meshes/collision/inner_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; visual mesh filename=../12345/Grippers/OnrobotRG2/visual/inner_knuckle.stl
- added link left_outer_knuckle, mass 0.05; collision mesh filename=package://onrobot_rg2_visualization/meshes/collision/outer_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; visual mesh filename=../12345/Grippers/OnrobotRG2/visual/outer_knuckle.stl
- added link onrobot_rg2_base_link, mass 0.7; collision mesh filename=package://onrobot_rg2_visualization/meshes/collision/base_l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; visual mesh filename=../12345/Grippers/OnrobotRG2/visual/base_link.stl
- added link right_inner_finger, mass 0.05; collision mesh filename=package://onrobot_rg2_visualization/meshes/collision/inner_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; visual mesh filename=../12345/Grippers/OnrobotRG2/visual/inner_finger.stl
- added link right_inner_knuckle, mass 0.05; collision mesh filename=package://onrobot_rg2_visualization/meshes/collision/inner_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; visual mesh filename=../12345/Grippers/OnrobotRG2/visual/inner_knuckle.stl
- added link right_outer_knuckle, mass 0.05; collision mesh filename=package://onrobot_rg2_visualization/meshes/collision/outer_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; visual mesh filename=../12345/Grippers/OnrobotRG2/visual/outer_knuckle.stl
Joints:
- added joint finger_joint: type revolute, parent onrobot_rg2_base_link, child left_outer_knuckle, origin xyz=0 -0.017178 0.125797 rpy=0 0 0, axis -1 0 0, limit lower=-0.558505 upper=0.785398 effort=1000 velocity=2.0
- added joint left_inner_finger_joint: type revolute, parent left_outer_knuckle, child left_inner_finger, origin xyz=0 -0.039592 0.038177000000000016 rpy=0 0 0, axis 1 0 0, limit lower=-0.872665 upper=0.872665 effort=1000 velocity=2.0, mimic joint=finger_joint multiplier=1 offset=0
- added joint left_inner_knuckle_joint: type revolute, parent onrobot_rg2_base_link, child left_inner_knuckle, origin xyz=0 -0.007678 0.1422970 rpy=0 0 0.0, axis 1 0 0, limit lower=-0.558505 upper=0.785398 effort=1000 velocity=2.0, mimic joint=finger_joint multiplier=-1 offset=0
- added joint right_inner_finger_joint: type revolute, parent right_outer_knuckle, child right_inner_finger, origin xyz=0 -0.039592 0.038177000000000016 rpy=0 0 0, axis 1 0 0, limit lower=-0.872665 upper=0.872665 effort=1000 velocity=2.0, mimic joint=finger_joint multiplier=1 offset=0
- added joint right_inner_knuckle_joint: type revolute, parent onrobot_rg2_base_link, child right_inner_knuckle, origin xyz=0 0.007678 0.1422970 rpy=0 0 -3.141592653589793, axis 1 0 0, limit lower=-0.558505 upper=0.785398 effort=1000 velocity=2.0, mimic joint=finger_joint multiplier=-1 offset=0
- added joint right_outer_knuckle_joint: type revolute, parent onrobot_rg2_base_link, child right_outer_knuckle, origin xyz=0 0.017178 0.125797 rpy=0 0 3.141592653589793, axis 1 0 0, limit lower=-0.558505 upper=0.785398 effort=1000 velocity=2.0, mimic joint=finger_joint multiplier=-1 offset=0
- added joint test: type fixed, parent base_link, child onrobot_rg2_base_link, origin xyz=0.3 0 0

Commit message: Update ScenarioC_Variant02.urdf

File: urdf/Scenario_C/ScenarioC_Variant02.urdf (robot description, URDF)
Before this commit: robot ur3_robot, 18 links, 17 joints
Joints:
- removed joint test
- joint flange-tool0: child tool0 -> onrobot_rg2_base_link

Commit message: Update ScenarioC_Variant02.urdf

File: urdf/Scenario_C/ScenarioC_Variant02.urdf (robot description, URDF)
Before this commit: robot ur3_robot, 18 links, 16 joints
Joints:
- added joint test: type fixed, parent base_link, child onrobot_rg2_base_link, origin xyz=0.3 0 0
- joint flange-tool0: child onrobot_rg2_base_link -> tool0

Commit message: Update ScenarioC_Variant02.urdf

File: urdf/Scenario_C/ScenarioC_Variant02.urdf (robot description, URDF)
Before this commit: robot ur3_robot, 18 links, 17 joints
Links:
- removed link tool0
Joints:
- removed joint test
- joint flange-tool0: child tool0 -> onrobot_rg2_base_link

Commit message: Update ScenarioC_Variant02.urdf

File: urdf/Scenario_C/ScenarioC_Variant02.urdf (robot description, URDF)
Before this commit: robot ur5, 19 links, 18 joints
Links:
- added link Slotted_Plate_Bench_700x720x900; visual mesh filename=../12345/Workstations/Slotted_Plate_Bench_700x720x900.stl
Joints:
- joint world_joint: origin xyz=0.0 0.0 0.0 rpy=0.0 0.0 0.0 -> xyz=0.0 0.0 0.9 rpy=0.0 0.0 0.0; parent world -> Slotted_Plate_Bench_700x720x900

Commit message: Update ScenarioC_Variant02.urdf

File: urdf/Scenario_C/ScenarioC_Variant02.urdf (robot description, URDF)
Before this commit: robot ur5, 20 links, 18 joints
Joints:
- removed joint world_joint
- added joint BenchToBaseLink_joint: type fixed, parent Slotted_Plate_Bench_700x720x900, child base_link, origin xyz=0.0 0.5 0.9 rpy=0.0 0.0 0.0
- added joint worldToBench_joint: type fixed, parent world, child Slotted_Plate_Bench_700x720x900, origin xyz=0.0 0.0 0.0 rpy=0.0 0.0 0.0

Commit message: Update ScenarioC_Variant02.urdf

File: urdf/Scenario_C/ScenarioC_Variant02.urdf (robot description, URDF)
Before this commit: robot ur5, 20 links, 19 joints
Joints:
- joint worldToBench_joint: origin xyz=0.0 0.0 0.0 rpy=0.0 0.0 0.0 -> xyz=2.0 0.0 0.0 rpy=0.0 0.0 0.0

Commit message: Update ScenarioC_Variant02.urdf

File: urdf/Scenario_C/ScenarioC_Variant02.urdf (robot description, URDF)
Before this commit: robot ur5, 20 links, 19 joints
Links:
- removed link world
- added link mybase_link, mass 4.0; collision mesh filename=package://ur_description/meshes/ur5/collision/base.stl; visual mesh filename=../12345/UR5/base.dae
- link base_link: mass 4.0 -> None; geometry visual cylinder length=1 radius=0.02
Joints:
- joint BenchToBaseLink_joint: child base_link -> mybase_link; origin xyz=0.0 0.5 0.9 rpy=0.0 0.0 0.0 -> xyz=0.5 0.5 0.919 rpy=0.0 0.0 -1.5708
- joint base_link-base_fixed_joint: parent base_link -> mybase_link
- joint shoulder_pan_joint: parent base_link -> mybase_link
- joint worldToBench_joint: origin xyz=2.0 0.0 0.0 rpy=0.0 0.0 0.0 -> xyz=1.0 0.0 0 rpy=0.0 0.0 0.0; parent world -> base_link

Commit message: Update ScenarioC_Variant02.urdf

File: urdf/Scenario_C/ScenarioC_Variant02.urdf (robot description, URDF)
Before this commit: robot ur5, 20 links, 19 joints
Links:
- removed link OnrobotSoftgripper
- added link OnrobotScrewdriver; visual mesh filename=../12345/Grippers/OnrobotScrewdriver/visual/OnRobotScrewdri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 scale=1 1 1
Joints:
- joint onrobot_Softgripper_DualQuickChanger_joint: child OnrobotSoftgripper -> OnrobotScrewdriver; origin xyz=-0.0465 0 0.0638 rpy=0 -1.047 0 -> xyz=-0.0435 0 0.0608 rpy=1.5708 -2.0944 3.1416
