Commit message: Update OnrobotSG_b.urdf

File: meshes/Grippers/OnrobotSoftgripper/OnrobotSG_b.urdf (robot description, URDF)
Before this commit: robot sg-b, 1 links, 0 joints
Links:
- link OnrobotSoftgripper: geometry collision cylinder length=0.10 radius=0.049; visual mesh filename=../12345/Grippers/OnrobotSoftgripper/visual/SG-b_v1.dae scale=1 1 1

Commit message: Update OnrobotSG_b.urdf

File: meshes/Grippers/OnrobotSoftgripper/OnrobotSG_b.urdf (robot description, URDF)
Before this commit: robot sg-b, 1 links, 0 joints
Links:
- added link base_link; visual cylinder length=1 radius=0.02
Joints:
- added joint test: type fixed, parent base_link, child OnrobotSoftgripper, origin xyz=0.3 0 0
