Commit message: Update OnrobotDualChangeWithRG2.urdf

File: meshes/Grippers/OnrobotDualQuickChanger/OnrobotDualChangeWithRG2.urdf (robot description, URDF)
Before this commit: robot onrobot_rg2_model, 8 links, 7 joints
Links:
- added link OnrobotDualQuickChanger_link; visual mesh filename=../12345/Grippers/OnrobotDualQuickChanger/visual/OnRobotDua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
Joints:
- removed joint test
- added joint OnrobotDualQuickChanger_base_joint: type fixed, parent base_link, child OnrobotDualQuickChanger_link, origin xyz=0.3 0 0
- added joint onrobot_rg2_DualQuickChanger_joint: type fixed, parent OnrobotDualQuickChanger_link, child onrobot_rg2_base_link, origin xyz=0.0336 0 0.0549 rpy=0 1.047 0

Commit message: Update OnrobotDualChangeWithRG2.urdf

File: meshes/Grippers/OnrobotDualQuickChanger/OnrobotDualChangeWithRG2.urdf (robot description, URDF)
Before this commit: robot onrobot_rg2_model, 9 links, 8 joints
Links:
- added link OnrobotSoftgripper, mass 0.001; collision cylinder length=0.10 radius=0.049; visual mesh filename=../12345/Grippers/OnrobotSoftgripper/visual/SG-b_v1.dae scale=1 1 1
Joints:
- joint onrobot_rg2_DualQuickChanger_joint: child onrobot_rg2_base_link -> OnrobotSoftgripper; origin xyz=0.0336 0 0.0549 rpy=0 1.047 0 -> xyz=-0.0336 0 0.0549 rpy=0 -1.047 0

Commit message: Update OnrobotDualChangeWithRG2.urdf

File: meshes/Grippers/OnrobotDualQuickChanger/OnrobotDualChangeWithRG2.urdf (robot description, URDF)
Before this commit: robot onrobot_rg2_model, 10 links, 8 joints
Links:
- removed link OnrobotDualQuickChanger_link
- removed link left_inner_finger
- removed link left_inner_knuckle
- removed link left_outer_knuckle
- removed link onrobot_rg2_base_link
- removed link right_inner_finger
- removed link right_inner_knuckle
- removed link right_outer_knuckle
Joints:
- removed joint OnrobotDualQuickChanger_base_joint
- removed joint finger_joint
- removed joint left_inner_finger_joint
- removed joint left_inner_knuckle_joint
- removed joint onrobot_rg2_DualQuickChanger_joint
- removed joint right_inner_finger_joint
- removed joint right_inner_knuckle_joint
- removed joint right_outer_knuckle_joint
- added joint test: type fixed, parent base_link, child OnrobotSoftgripper, origin xyz=0.3 0 0

Commit message: Update OnrobotDualChangeWithRG2.urdf

File: meshes/Grippers/OnrobotDualQuickChanger/OnrobotDualChangeWithRG2.urdf (robot description, URDF)
Before this commit: robot sg-b, 2 links, 1 joints
Links:
- added link OnrobotDualQuickChanger_link; visual mesh filename=../12345/Grippers/OnrobotDualQuickChanger/visual/OnRobotDua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
- added link left_inner_finger, mass 0.05; collision mesh filename=package://onrobot_rg2_visualization/meshes/collision/inner_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; visual mesh filename=../12345/Grippers/OnrobotRG2/visual/inner_finger.stl
- added link left_inner_knuckle, mass 0.05; collision mesh filename=package://onrobot_rg2_visualization/meshes/collision/inner_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; visual mesh filename=../12345/Grippers/OnrobotRG2/visual/inner_knuckle.stl
- added link left_outer_knuckle, mass 0.05; collision mesh filename=package://onrobot_rg2_visualization/meshes/collision/outer_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; visual mesh filename=../12345/Grippers/OnrobotRG2/visual/outer_knuckle.stl
- added link onrobot_rg2_base_link, mass 0.7; collision mesh filename=package://onrobot_rg2_visualization/meshes/collision/base_l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; visual mesh filename=../12345/Grippers/OnrobotRG2/visual/base_link.stl
- added link right_inner_finger, mass 0.05; collision mesh filename=package://onrobot_rg2_visualization/meshes/collision/inner_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; visual mesh filename=../12345/Grippers/OnrobotRG2/visual/inner_finger.stl
- added link right_inner_knuckle, mass 0.05; collision mesh filename=package://onrobot_rg2_visualization/meshes/collision/inner_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; visual mesh filename=../12345/Grippers/OnrobotRG2/visual/inner_knuckle.stl
- added link right_outer_knuckle, mass 0.05; collision mesh filename=package://onrobot_rg2_visualization/meshes/collision/outer_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; visual mesh filename=../12345/Grippers/OnrobotRG2/visual/outer_knuckle.stl
Joints:
- removed joint test
- added joint OnrobotDualQuickChanger_base_joint: type fixed, parent base_link, child OnrobotDualQuickChanger_link, origin xyz=0.3 0 0
- added joint finger_joint: type revolute, parent onrobot_rg2_base_link, child left_outer_knuckle, origin xyz=0 -0.017178 0.125797 rpy=0 0 0, axis -1 0 0, limit lower=-0.558505 upper=0.785398 effort=1000 velocity=2.0
- added joint left_inner_finger_joint: type revolute, parent left_outer_knuckle, child left_inner_finger, origin xyz=0 -0.039592 0.038177000000000016 rpy=0 0 0, axis 1 0 0, limit lower=-0.872665 upper=0.872665 effort=1000 velocity=2.0, mimic joint=finger_joint multiplier=1 offset=0
- added joint left_inner_knuckle_joint: type revolute, parent onrobot_rg2_base_link, child left_inner_knuckle, origin xyz=0 -0.007678 0.1422970 rpy=0 0 0.0, axis 1 0 0, limit lower=-0.558505 upper=0.785398 effort=1000 velocity=2.0, mimic joint=finger_joint multiplier=-1 offset=0
- added joint onrobot_rg2_DualQuickChanger_joint: type fixed, parent OnrobotDualQuickChanger_link, child OnrobotSoftgripper, origin xyz=-0.0465 0 0.0638 rpy=0 -1.047 0
- added joint right_inner_finger_joint: type revolute, parent right_outer_knuckle, child right_inner_finger, origin xyz=0 -0.039592 0.038177000000000016 rpy=0 0 0, axis 1 0 0, limit lower=-0.872665 upper=0.872665 effort=1000 velocity=2.0, mimic joint=finger_joint multiplier=1 offset=0
- added joint right_inner_knuckle_joint: type revolute, parent onrobot_rg2_base_link, child right_inner_knuckle, origin xyz=0 0.007678 0.1422970 rpy=0 0 -3.141592653589793, axis 1 0 0, limit lower=-0.558505 upper=0.785398 effort=1000 velocity=2.0, mimic joint=finger_joint multiplier=-1 offset=0
- added joint right_outer_knuckle_joint: type revolute, parent onrobot_rg2_base_link, child right_outer_knuckle, origin xyz=0 0.017178 0.125797 rpy=0 0 3.141592653589793, axis 1 0 0, limit lower=-0.558505 upper=0.785398 effort=1000 velocity=2.0, mimic joint=finger_joint multiplier=-1 offset=0

Commit message: Update OnrobotDualChangeWithRG2.urdf

File: meshes/Grippers/OnrobotDualQuickChanger/OnrobotDualChangeWithRG2.urdf (robot description, URDF)
Before this commit: robot onrobot_rg2_model, 10 links, 8 joints
Joints:
- added joint onrobot_Softgripper_DualQuickChanger_joint: type fixed, parent OnrobotDualQuickChanger_link, child OnrobotSoftgripper, origin xyz=-0.0465 0 0.0638 rpy=0 -1.047 0
- joint onrobot_rg2_DualQuickChanger_joint: child OnrobotSoftgripper -> onrobot_rg2_base_link; origin xyz=-0.0465 0 0.0638 rpy=0 -1.047 0 -> xyz=0.0336 0 0.0549 rpy=0 1.047 0
