Commit message: Update workstations.urdf

File: meshes/Workstations/workstations.urdf (robot description, URDF)
Before this commit: robot Workstations, 2 links, 1 joints
Links:
- added link conveyerTable; visual mesh filename=../12345/Workstations/transportband01.stl
Joints:
- added joint test: type fixed, parent base_link, child conveyerTable, origin xyz=0 2 0.9

Commit message: Update workstations.urdf

File: meshes/Workstations/workstations.urdf (robot description, URDF)
Before this commit: robot Workstations, 3 links, 2 joints
Links:
- link conveyerTable: geometry visual mesh filename=../12345/Workstations/transportband02.stl

Commit message: Update workstations.urdf

File: meshes/Workstations/workstations.urdf (robot description, URDF)
Before this commit: robot Workstations, 3 links, 2 joints
Links:
- link base_link: geometry visual cylinder length=1 radius=0.02
Joints:
- joint BenchTobaseLink: child UR10_Workbench -> Slottted_Plate_Bench_700x1500; origin xyz=0 2 0.9 -> xyz=2 1 0.9
- joint test: origin xyz=0 2 0.9 -> xyz=-3 2 0.9

Commit message: Update workstations.urdf

File: meshes/Workstations/workstations.urdf (robot description, URDF)
Before this commit: robot Workstations, 3 links, 2 joints
Links:
- removed link Slottted_Plate_Bench_700x1500
- added link Slotted_Plate_Bench_700x1500; visual mesh filename=../12345/Workstations/Slotted_Plate_Bench_700x1500.stl
- added link WoodPlate_Bench_700x1500x900; visual mesh filename=../12345/Workstations/WoodPlate_Bench_700x1500x900.stl
Joints:
- removed joint BenchTobaseLink
- added joint Slotted_Plate_Bench_700x1500TobaseLink: type fixed, parent base_link, child Slotted_Plate_Bench_700x1500, origin xyz=2 1 0.9
- added joint WoodPlate_Bench_700x1500x900TobaseLink: type fixed, parent base_link, child WoodPlate_Bench_700x1500x900, origin xyz=2 3 0.9

Commit message: Update workstations.urdf

File: meshes/Workstations/workstations.urdf (robot description, URDF)
Before this commit: robot Workstations, 4 links, 3 joints
Links:
- added link Stele_600x600x1015; visual mesh filename=../12345/Workstations/Stele_600x600x1015.stl
Joints:
- removed joint Slotted_Plate_Bench_700x1500TobaseLink
- removed joint WoodPlate_Bench_700x1500x900TobaseLink
- removed joint test
- added joint Slotted_Plate_Bench_700x1500ToBaseLink: type fixed, parent base_link, child Slotted_Plate_Bench_700x1500, origin xyz=2 1 0.9
- added joint Stele_600x600x1015ToBaseLink: type fixed, parent base_link, child Stele_600x600x1015, origin xyz=-3 2 0.9
- added joint WoodPlate_Bench_700x1500x900ToBaseLink: type fixed, parent base_link, child WoodPlate_Bench_700x1500x900, origin xyz=2 3 0.9
- added joint conveyerTableToBaseLink: type fixed, parent base_link, child conveyerTable, origin xyz=-3 1 0

Commit message: Update workstations.urdf

File: meshes/Workstations/workstations.urdf (robot description, URDF)
Before this commit: robot Workstations, 5 links, 4 joints
Joints:
- joint Stele_600x600x1015ToBaseLink: origin xyz=-3 2 0.9 -> xyz=-3 2 0
- joint conveyerTableToBaseLink: origin xyz=-3 1 0 -> xyz=-3 1 0.9

Commit message: Update workstations.urdf

File: meshes/Workstations/workstations.urdf (robot description, URDF)
Before this commit: robot Workstations, 5 links, 4 joints
Links:
- added link Slotted_Plate_Bench_700x720x900; visual mesh filename=../12345/Workstations/Slotted_Plate_Bench_700x720x900.stl
Joints:
- added joint Slotted_Plate_Bench_700x720x900ToBaseLink: type fixed, parent base_link, child Slotted_Plate_Bench_700x720x900, origin xyz=2 0 0

Commit message: Update workstations.urdf

File: meshes/Workstations/workstations.urdf (robot description, URDF)
Before this commit: robot Workstations, 6 links, 5 joints
Joints:
- joint Slotted_Plate_Bench_700x720x900ToBaseLink: origin xyz=2 0 0 -> xyz=2 -1 0
