Commit message: Update table.xacro

File: my_robot_description/urdf/table.xacro (robot description, xacro)
@@ -0,0 +1,26 @@
+<?xml version="1.0"?>
+<robot xmlns:xacro="http://www.ros.org/wiki/xacro" name="wood_table">
+  <!-- ========== TABLE MACRO ========== -->
+  <xacro:macro name="wood_table" params="name parent x y z">
+    <!-- Table base link -->
+    <link name="${name}_link">
+      <visual>
+        <geometry>
+          <mesh filename="package://my_robot_description/meshes/stl/WoodPlate_Bench_700x1500x900.stl"/>
+        </geometry>
+      </visual>
+      <collision>
+        <geometry>
+          <mesh filename="package://my_robot_description/meshes/stl/WoodPlate_Bench_700x1500x900.stl"/>
+        </geometry>
+      </collision>
+    </link>
+    <!-- Fixed joint to world or parent -->
+    <joint name="${name}_joint" type="fixed">
+      <parent link="${parent}"/>
+      <child link="${name}_link"/>
+      <!-- Position of table in world -->
+      <origin xyz="${x} ${y} ${z}" rpy="0 0 0"/>
+    </joint>
+  </xacro:macro>
+</robot>

Commit message: Update table.xacro

File: my_robot_description/urdf/table.xacro (robot description, xacro)
@@ -1,26 +1,18 @@
 <?xml version="1.0"?>
-<robot xmlns:xacro="http://www.ros.org/wiki/xacro" name="wood_table">
-  <!-- ========== TABLE MACRO ========== -->
-  <xacro:macro name="wood_table" params="name parent x y z">
-    <!-- Table base link -->
-    <link name="${name}_link">
-      <visual>
-        <geometry>
-          <mesh filename="package://my_robot_description/meshes/stl/WoodPlate_Bench_700x1500x900.stl"/>
-        </geometry>
-      </visual>
-      <collision>
-        <geometry>
-          <mesh filename="package://my_robot_description/meshes/stl/WoodPlate_Bench_700x1500x900.stl"/>
-        </geometry>
-      </collision>
-    </link>
-    <!-- Fixed joint to world or parent -->
-    <joint name="${name}_joint" type="fixed">
-      <parent link="${parent}"/>
-      <child link="${name}_link"/>
-      <!-- Position of table in world -->
-      <origin xyz="${x} ${y} ${z}" rpy="0 0 0"/>
-    </joint>
-  </xacro:macro>
+<robot xmlns:xacro="http://www.ros.org/wiki/xacro" name="table">
+  <link name="table_link">
+    <visual>
+      <geometry>
+        <mesh filename="package://my_robot_description/meshes/WoodPlate_Bench_700x1500x900.stl"/>
+      </geometry>
+      <material name="gray">
+        <color rgba="0.7 0.7 0.7 1.0"/>
+      </material>
+    </visual>
+    <collision>
+      <geometry>
+        <box size="1.5 0.7 0.05"/>
+      </geometry>
+    </collision>
+  </link>
 </robot>
