Commit message: Update ur5_with_gripper.xacro

File: my_robot_description/urdf/ur5_with_gripper.xacro (robot description, xacro)
@@ -17,5 +17,12 @@
   </joint>
   <!-- Left finger -->
-  <link name="finger_left_link"/>
+<link name="finger_left_link">
+  <visual>
+    <geometry>
+      <box size="0.02 0.01 0.08"/>
+    </geometry>
+    <material name="blue"/>
+  </visual>
+</link>
   <joint name="finger_left_joint" type="prismatic">
     <parent link="gripper_base_link"/>
@@ -25,5 +32,12 @@
   </joint>
   <!-- Right finger -->
-  <link name="finger_right_link"/>
+  <link name="finger_right_link">
+  <visual>
+    <geometry>
+      <box size="0.02 0.01 0.08"/>
+    </geometry>
+    <material name="red"/>
+  </visual>
+</link>
   <joint name="finger_right_joint" type="prismatic">
     <parent link="gripper_base_link"/>

Commit message: Update ur5_with_gripper.xacro

File: my_robot_description/urdf/ur5_with_gripper.xacro (robot description, xacro)
@@ -37,5 +37,7 @@
       <box size="0.02 0.01 0.08"/>
     </geometry>
-    <material name="red"/>
+    <material name="rightFinger" >
+    <color rgba ="0.5020 0.0000 0.5020 1"/>
+    </material>
   </visual>
 </link>

Commit message: Update ur5_with_gripper.xacro

File: my_robot_description/urdf/ur5_with_gripper.xacro (robot description, xacro)
@@ -22,5 +22,7 @@
       <box size="0.02 0.01 0.08"/>
     </geometry>
-    <material name="blue"/>
+    <material name="leftFinger" >
+    <color rgba ="1 0 0 1"/>
+    </material>
   </visual>
 </link>

Commit message: Update ur5_with_gripper.xacro

File: my_robot_description/urdf/ur5_with_gripper.xacro (robot description, xacro)
@@ -10,9 +10,18 @@
   <!-- ===================== -->
   <!-- Gripper base attached to tool0 -->
-  <link name="gripper_base_link"/>
+  <link name="gripper_base_link">
+  <visual>
+    <geometry>
+      <box size="0.01 0.01 0.01"/>
+    </geometry>
+    <material name="gripperbase" >
+    <color rgba ="1 0 1 1"/>
+    </material>
+  </visual>
+</link>
   <joint name="tool0_to_gripper" type="fixed">
     <parent link="tool0"/>
     <child link="gripper_base_link"/>
-    <origin xyz="0 0 0" rpy="0 0 0"/>
+    <origin xyz="0 0 0.1" rpy="0 0 0"/>
   </joint>
   <!-- Left finger -->

Commit message: Update ur5_with_gripper.xacro

File: my_robot_description/urdf/ur5_with_gripper.xacro (robot description, xacro)
@@ -29,5 +29,5 @@
   <visual>
     <geometry>
-      <box size="0.02 0.01 0.08"/>
+      <box size="0.1 0.1 0.1"/>
     </geometry>
     <material name="leftFinger" >
@@ -46,5 +46,5 @@
   <visual>
     <geometry>
-      <box size="0.02 0.01 0.08"/>
+      <box size="0.1 0.1 0.1"/>
     </geometry>
     <material name="rightFinger" >

Commit message: Update ur5_with_gripper.xacro

File: my_robot_description/urdf/ur5_with_gripper.xacro (robot description, xacro)
@@ -39,4 +39,5 @@
     <parent link="gripper_base_link"/>
     <child link="finger_left_link"/>
+    <origin xyz="0 0.05 0" rpy="0 0 0"/>
     <axis xyz="1 0 0"/>
     <limit effort="10" velocity="0.1" lower="0.0" upper="0.04"/>
@@ -45,9 +46,10 @@
   <link name="finger_right_link">
   <visual>
+  <origin xyz="0 -0.05 0" rpy="0 0 0"/>
     <geometry>
       <box size="0.1 0.1 0.1"/>
     </geometry>
     <material name="rightFinger" >
-    <color rgba ="0 0 1 1"/>
+    <color rgba ="0 0 1 0.5"/>
     </material>
   </visual>

Commit message: Update ur5_with_gripper.xacro

File: my_robot_description/urdf/ur5_with_gripper.xacro (robot description, xacro)
@@ -13,5 +13,5 @@
   <visual>
     <geometry>
-      <box size="0.01 0.01 0.01"/>
+      <box size="0.05 0.05 0.05"/>
     </geometry>
     <material name="gripperbase" >
@@ -28,8 +28,9 @@
 <link name="finger_left_link">
   <visual>
+ <origin xyz="0 0 0" rpy="0 0 0"/>
     <geometry>
-      <box size="0.1 0.1 0.1"/>
+       <box size="0.05 0.05 0.1"/>
     </geometry>
-    <material name="leftFinger" >
+    <material name="leftFingerGreen" >
     <color rgba ="0 1 0 1"/>
     </material>
@@ -39,5 +40,5 @@
     <parent link="gripper_base_link"/>
     <child link="finger_left_link"/>
-    <origin xyz="0 0.05 0" rpy="0 0 0"/>
+    <origin xyz="0 0.05 0.1" rpy="0 0 0"/>
     <axis xyz="1 0 0"/>
     <limit effort="10" velocity="0.1" lower="0.0" upper="0.04"/>
@@ -46,9 +47,9 @@
   <link name="finger_right_link">
   <visual>
-  <origin xyz="0 -0.05 0" rpy="0 0 0"/>
+  <origin xyz="0 0 0" rpy="0 0 0"/>
     <geometry>
-      <box size="0.1 0.1 0.1"/>
+      <box size="0.05 0.05 0.1"/>
     </geometry>
-    <material name="rightFinger" >
+    <material name="rightFingerBlue" >
     <color rgba ="0 0 1 0.5"/>
     </material>
@@ -58,4 +59,5 @@
     <parent link="gripper_base_link"/>
     <child link="finger_right_link"/>
+    <origin xyz="0 -0.05 0.1" rpy="0 0 0"/>
     <axis xyz="-1 0 0"/>
     <limit effort="10" velocity="0.1" lower="0.0" upper="0.04"/>

Commit message: Update ur5_with_gripper.xacro

File: my_robot_description/urdf/ur5_with_gripper.xacro (robot description, xacro)
@@ -6,60 +6,9 @@
   <xacro:include filename="$(find ur_description)/urdf/inc/ur5_macro.xacro"/>
   <xacro:ur5_robot prefix="" />
+ <!-- ===================== -->
+  <!-- INCLUDE GRIPPER       -->
   <!-- ===================== -->
-  <!-- GRIPPER ADDITION      -->
-  <!-- ===================== -->
-  <!-- Gripper base attached to tool0 -->
-  <link name="gripper_base_link">
-  <visual>
-    <geometry>
-      <box size="0.05 0.05 0.05"/>
-    </geometry>
-    <material name="gripperbase" >
-    <color rgba ="1 0 1 1"/>
-    </material>
-  </visual>
-</link>
-  <joint name="tool0_to_gripper" type="fixed">
-    <parent link="tool0"/>
-    <child link="gripper_base_link"/>
-    <origin xyz="0 0 0.1" rpy="0 0 0"/>
-  </joint>
-  <!-- Left finger -->
-<link name="finger_left_link">
-  <visual>
- <origin xyz="0 0 0" rpy="0 0 0"/>
-    <geometry>
-       <box size="0.05 0.05 0.1"/>
-    </geometry>
-    <material name="leftFingerGreen" >
-    <color rgba ="0 1 0 1"/>
-    </material>
-  </visual>
-</link>
-  <joint name="finger_left_joint" type="prismatic">
-    <parent link="gripper_base_link"/>
-    <child link="finger_left_link"/>
-    <origin xyz="0 0.05 0.1" rpy="0 0 0"/>
-    <axis xyz="1 0 0"/>
-    <limit effort="10" velocity="0.1" lower="0.0" upper="0.04"/>
-  </joint>
-  <!-- Right finger -->
-  <link name="finger_right_link">
-  <visual>
-  <origin xyz="0 0 0" rpy="0 0 0"/>
-    <geometry>
-      <box size="0.05 0.05 0.1"/>
-    </geometry>
-    <material name="rightFingerBlue" >
-    <color rgba ="0 0 1 0.5"/>
-    </material>
-  </visual>
-</link>
-  <joint name="finger_right_joint" type="prismatic">
-    <parent link="gripper_base_link"/>
-    <child link="finger_right_link"/>
-    <origin xyz="0 -0.05 0.1" rpy="0 0 0"/>
-    <axis xyz="-1 0 0"/>
-    <limit effort="10" velocity="0.1" lower="0.0" upper="0.04"/>
-  </joint>
+  <xacro:include filename="$(find your_package)/urdf/MyFingerGrip.xacro"/>
+  <!-- Attach gripper to tool0 -->
+  <xacro:MyFingerGrip parent="tool0"/>
 </robot>

Commit message: Update ur5_with_gripper.xacro

File: my_robot_description/urdf/ur5_with_gripper.xacro (robot description, xacro)
@@ -4,10 +4,29 @@
   <!-- UR5 BASE ROBOT        -->
   <!-- ===================== -->
-  <xacro:include filename="$(find my_robot_description)/urdf/inc/ur5_macro.xacro"/>
+  <xacro:include filename="$(find ur_description)/urdf/inc/ur5_macro.xacro"/>
   <xacro:ur5_robot prefix="" />
+  <!-- ===================== -->
+  <!-- GRIPPER ADDITION      -->
+  <!-- ===================== -->
+  <!-- Gripper base attached to tool0 -->
+  <link name="1gripper_base_link">
+  <visual>
+    <geometry>
+      <box size="0.05 0.05 0.05"/>
+    </geometry>
+    <material name="gripperbase" >
+    <color rgba ="1 0 1 1"/>
+    </material>
+  </visual>
+</link>
+  <joint name="tool0_to_gripper" type="fixed">
+    <parent link="tool0"/>
+    <child link="1gripper_base_link"/>
+    <origin xyz="0 0 0.1" rpy="0 0 0"/>
+  </joint>
  <!-- ===================== -->
   <!-- INCLUDE GRIPPER       -->
   <!-- ===================== -->
-  <xacro:include filename="$(find your_package)/urdf/MyFingerGrip.xacro"/>
+  <xacro:include filename="$(find my_robot_description)/urdf/MyFingerGrip.xacro"/>
   <!-- Attach gripper to tool0 -->
   <xacro:MyFingerGrip parent="tool0"/>

Commit message: Update ur5_with_gripper.xacro

File: my_robot_description/urdf/ur5_with_gripper.xacro (robot description, xacro)
@@ -9,25 +9,6 @@
   <!-- GRIPPER ADDITION      -->
   <!-- ===================== -->
-  <!-- Gripper base attached to tool0 -->
-  <link name="1gripper_base_link">
-  <visual>
-    <geometry>
-      <box size="0.05 0.05 0.05"/>
-    </geometry>
-    <material name="gripperbase" >
-    <color rgba ="1 0 1 1"/>
-    </material>
-  </visual>
-</link>
-  <joint name="tool0_to_gripper" type="fixed">
-    <parent link="tool0"/>
-    <child link="1gripper_base_link"/>
-    <origin xyz="0 0 0.1" rpy="0 0 0"/>
-  </joint>
- <!-- ===================== -->
-  <!-- INCLUDE GRIPPER       -->
-  <!-- ===================== -->
   <xacro:include filename="$(find my_robot_description)/urdf/MyFingerGrip.xacro"/>
-  <!-- Attach gripper to tool0 -->
+  <!-- Attach gripper to tool0  this is default name of rosindustrial UR connection link -->
   <xacro:MyFingerGrip parent="tool0"/>
 </robot>
