Commit message: Update MyFingerGrip.xacro

File: my_robot_description/urdf/MyFingerGrip.xacro (robot description, xacro)
@@ -0,0 +1,69 @@
+<?xml version="1.0"?>
+<robot xmlns:xacro="http://www.ros.org/wiki/xacro">
+  <xacro:macro name="simple_gripper" params="parent">
+    <!-- ===================== -->
+    <!-- GRIPPER BASE          -->
+    <!-- ===================== -->
+    <link name="gripper_base_link">
+      <visual>
+        <geometry>
+          <box size="0.05 0.05 0.05"/>
+        </geometry>
+        <material name="gripperbase">
+          <color rgba="1 0 1 1"/>
+        </material>
+      </visual>
+    </link>
+    <joint name="tool0_to_gripper" type="fixed">
+      <parent link="${parent}"/>
+      <child link="gripper_base_link"/>
+      <origin xyz="0 0 0.1" rpy="0 0 0"/>
+    </joint>
+    <!-- ===================== -->
+    <!-- LEFT FINGER           -->
+    <!-- ===================== -->
+    <link name="finger_left_link">
+      <visual>
+        <geometry>
+          <box size="0.05 0.05 0.1"/>
+        </geometry>
+        <material name="leftFingerGreen">
+          <color rgba="0 1 0 1"/>
+        </material>
+      </visual>
+    </link>
+    <joint name="finger_left_joint" type="prismatic">
+      <parent link="gripper_base_link"/>
+      <child link="finger_left_link"/>
+      <origin xyz="0 0.05 0.1" rpy="0 0 0"/>
+      <axis xyz="1 0 0"/>
+      <limit lower="0.0"
+             upper="0.04"
+             effort="10"
+             velocity="0.1"/>
+    </joint>
+    <!-- ===================== -->
+    <!-- RIGHT FINGER          -->
+    <!-- ===================== -->
+    <link name="finger_right_link">
+      <visual>
+        <geometry>
+          <box size="0.05 0.05 0.1"/>
+        </geometry>
+        <material name="rightFingerBlue">
+          <color rgba="0 0 1 0.5"/>
+        </material>
+      </visual>
+    </link>
+    <joint name="finger_right_joint" type="prismatic">
+      <parent link="gripper_base_link"/>
+      <child link="finger_right_link"/>
+      <origin xyz="0 -0.05 0.1" rpy="0 0 0"/>
+      <axis xyz="-1 0 0"/>
+      <limit lower="0.0"
+             upper="0.04"
+             effort="10"
+             velocity="0.1"/>
+    </joint>
+  </xacro:macro>
+</robot>

Commit message: Update MyFingerGrip.xacro

File: my_robot_description/urdf/MyFingerGrip.xacro (robot description, xacro)
@@ -1,8 +1,6 @@
 <?xml version="1.0"?>
 <robot xmlns:xacro="http://www.ros.org/wiki/xacro">
-  <xacro:macro name="simple_gripper" params="parent">
-    <!-- ===================== -->
-    <!-- GRIPPER BASE          -->
-    <!-- ===================== -->
+  <xacro:macro name="MyFingerGrip" params="parent">
+     <!-- GRIPPER BASE          -->
     <link name="gripper_base_link">
       <visual>
@@ -20,9 +18,8 @@
       <origin xyz="0 0 0.1" rpy="0 0 0"/>
     </joint>
-    <!-- ===================== -->
     <!-- LEFT FINGER           -->
-    <!-- ===================== -->
     <link name="finger_left_link">
       <visual>
+      <origin xyz="0 0 0" rpy="0 0 0"/>
         <geometry>
           <box size="0.05 0.05 0.1"/>
@@ -38,14 +35,10 @@
       <origin xyz="0 0.05 0.1" rpy="0 0 0"/>
       <axis xyz="1 0 0"/>
-      <limit lower="0.0"
-             upper="0.04"
-             effort="10"
-             velocity="0.1"/>
+      <limit lower="0.0" upper="0.04" effort="10" velocity="0.1"/>
     </joint>
-    <!-- ===================== -->
     <!-- RIGHT FINGER          -->
-    <!-- ===================== -->
     <link name="finger_right_link">
       <visual>
+       <origin xyz="0 0 0" rpy="0 0 0"/>
         <geometry>
           <box size="0.05 0.05 0.1"/>
@@ -61,8 +54,5 @@
       <origin xyz="0 -0.05 0.1" rpy="0 0 0"/>
       <axis xyz="-1 0 0"/>
-      <limit lower="0.0"
-             upper="0.04"
-             effort="10"
-             velocity="0.1"/>
+      <limit lower="0.0" upper="0.04" effort="10" velocity="0.1"/>
     </joint>
   </xacro:macro>

Commit message: Update MyFingerGrip.xacro

File: my_robot_description/urdf/MyFingerGrip.xacro (robot description, xacro)
@@ -12,4 +12,11 @@
         </material>
       </visual>
+      <!-- COLLISION -->
+      <collision>
+        <origin xyz="0 0 0" rpy="0 0 0"/>
+        <geometry>
+          <box size="0.05 0.05 0.05"/>
+        </geometry>
+      </collision>
     </link>
     <joint name="tool0_to_gripper" type="fixed">

Commit message: Update MyFingerGrip.xacro

File: my_robot_description/urdf/MyFingerGrip.xacro (robot description, xacro)
@@ -36,4 +36,11 @@
         </material>
       </visual>
+  <!-- COLLISION -->
+      <collision>
+        <origin xyz="0 0 0" rpy="0 0 0"/>
+        <geometry>
+           <box size="0.05 0.05 0.1"/>
+        </geometry>
+      </collision>
     </link>
     <joint name="finger_left_joint" type="prismatic">
@@ -55,4 +62,11 @@
         </material>
       </visual>
+ <!-- COLLISION -->
+      <collision>
+        <origin xyz="0 0 0" rpy="0 0 0"/>
+        <geometry>
+          <box size="0.05 0.05 0.1"/>
+        </geometry>
+      </collision>
     </link>
     <joint name="finger_right_joint" type="prismatic">
