Commit message: Update robot.xacro

File: my_robot_description/urdf/robot.xacro (robot description, xacro)
@@ -1,4 +1,16 @@
 <?xml version="1.0"?>
 <robot xmlns:xacro="http://www.ros.org/wiki/xacro" name="robot">
+ <!-- Base link -->
+  <link name="base_link">
+    <visual>
+      <origin xyz="0 0 ${link_height_offset}" rpy="0 0 0"/>
+      <geometry>
+        <cylinder radius="${link_radius}" length="${link_length}"/>
+      </geometry>
+      <material name="green">
+        <color rgba="0 1 0 1"/>
+      </material>
+    </visual>
+  </link>
   <!-- Table dimensions -->
   <xacro:property name="table_length" value="1.2"/>
@@ -32,3 +44,9 @@
     </inertial>
   </link>
+  <!-- connect UR base to bench -->
+  <joint name="base_to_table" type="fixed">
+    <parent link="base_link"/>
+    <child link="table_link"/>
+    <origin xyz="1 0 0" rpy="0 0 0"/>
+  </joint>
 </robot>

Commit message: Update robot.xacro

File: my_robot_description/urdf/robot.xacro (robot description, xacro)
@@ -1,5 +1,6 @@
 <?xml version="1.0"?>
-<robot xmlns:xacro="http://www.ros.org/wiki/xacro" name="robot">
- <!-- Base link -->
+<robot xmlns:xacro="http://www.ros.org/wiki/xacro" name="my_robot">
+   <!-- include UR robot -->
+  <xacro:include filename="$(find ur_description)/urdf/ur5_robot.urdf.xacro"/>
   <link name="base_link">
     <visual>
@@ -9,44 +10,24 @@
       </geometry>
       <material name="green">
-        <color rgba="0 1 0 1"/>
-      </material>
-    </visual>
-  </link>
-  <!-- Table dimensions -->
-  <xacro:property name="table_length" value="1.2"/>
-  <xacro:property name="table_width" value="0.8"/>
-  <xacro:property name="table_height" value="0.75"/>
-  <xacro:property name="table_thickness" value="0.05"/>
-  <!-- Main table link -->
-  <link name="table_link">
-    <visual>
-      <geometry>
-        <box size="${table_length} ${table_width} ${table_thickness}"/>
-      </geometry>
-      <origin xyz="0 1 ${table_height}" rpy="0 0 0"/>
-      <material name="brown">
-        <color rgba="0 0 1 1"/>
+        <color rgba="1 0 0 1"/>
       </material>
     </visual>
     <collision>
+      <origin xyz="0 0 ${link_height_offset}" rpy="0 0 0"/>
       <geometry>
-        <box size="${table_length} ${table_width} ${table_thickness}"/>
+        <cylinder radius="${link_radius}" length="${link_length}"/>
       </geometry>
-      <origin xyz="0 1 ${table_height}" rpy="0 0 0"/>
     </collision>
     <inertial>
-      <origin xyz="0 0 ${table_height}" rpy="0 0 0"/>
-      <mass value="20.0"/>
-      <inertia
-        ixx="1.0" ixy="0.0" ixz="0.0"
-        iyy="1.0" iyz="0.0"
-        izz="1.0"/>
+      <origin xyz="0 0 ${link_height_offset}" rpy="0 0 0"/>
+      <mass value="5.0"/>
+      <inertia ixx="0.1" ixy="0.0" ixz="0.0"
+               iyy="0.1" iyz="0.0"
+               izz="0.1"/>
     </inertial>
   </link>
-  <!-- connect UR base to bench -->
-  <joint name="base_to_table" type="fixed">
+  <joint name="table_to_ur5" type="fixed">
     <parent link="base_link"/>
-    <child link="table_link"/>
-    <origin xyz="1 0 0" rpy="0 0 0"/>
+    <child link="ur5_base_link"/>
   </joint>
 </robot>

Commit message: Update robot.xacro

File: my_robot_description/urdf/robot.xacro (robot description, xacro)
@@ -1,6 +1,8 @@
 <?xml version="1.0"?>
 <robot xmlns:xacro="http://www.ros.org/wiki/xacro" name="my_robot">
-   <!-- include UR robot -->
-  <xacro:include filename="$(find ur_description)/urdf/ur5_robot.urdf.xacro"/>
+  <!-- Base cylinder -->
+ <xacro:property name="link_radius" value="0.02"/>
+  <xacro:property name="link_length" value="3.0"/>
+  <xacro:property name="link_height_offset" value="0.5"/>
   <link name="base_link">
     <visual>
@@ -27,7 +29,3 @@
     </inertial>
   </link>
-  <joint name="table_to_ur5" type="fixed">
-    <parent link="base_link"/>
-    <child link="ur5_base_link"/>
-  </joint>
 </robot>

Commit message: Update robot.xacro

File: my_robot_description/urdf/robot.xacro (robot description, xacro)
@@ -1,2 +1,40 @@
+<?xml version="1.0"?>
+<robot xmlns:xacro="http://www.ros.org/wiki/xacro" name="my_robot">
+ <xacro:include filename="$(find ur_description)/urdf/inc/ur5_macro.xacro"/>
+  <xacro:ur5_robot prefix="ur5_" />
+  <!-- Base cylinder -->
+ <xacro:property name="link_radius" value="0.02"/>
+  <xacro:property name="link_length" value="3.0"/>
+  <xacro:property name="link_height_offset" value="0.5"/>
+  <link name="base_link">
+    <visual>
+      <origin xyz="0 0 ${link_height_offset}" rpy="0 0 0"/>
+      <geometry>
+        <cylinder radius="${link_radius}" length="${link_length}"/>
+      </geometry>
+      <material name="green">
+        <color rgba="1 0 0 1"/>
+      </material>
+    </visual>
+    <collision>
+      <origin xyz="0 0 ${link_height_offset}" rpy="0 0 0"/>
+      <geometry>
+        <cylinder radius="${link_radius}" length="${link_length}"/>
+      </geometry>
+    </collision>
+    <inertial>
+      <origin xyz="0 0 ${link_height_offset}" rpy="0 0 0"/>
+      <mass value="5.0"/>
+      <inertia ixx="0.1" ixy="0.0" ixz="0.0"
+               iyy="0.1" iyz="0.0"
+               izz="0.1"/>
+    </inertial>
+  </link>
+ <joint name="base_to_table" type="fixed">
+    <parent link="base_link"/>
+    <child link="ur5_base_link"/>
+    <origin xyz="0 1 0.9" rpy="0 0 0"/>
+  </joint>
+</robot>
 <?xml version="1.0"?>
 <robot xmlns:xacro="http://www.ros.org/wiki/xacro" name="my_robot">

Commit message: Update robot.xacro

File: my_robot_description/urdf/robot.xacro (robot description, xacro)
@@ -1,10 +1,10 @@
 <?xml version="1.0"?>
 <robot xmlns:xacro="http://www.ros.org/wiki/xacro" name="my_robot">
+  <!-- Base cylinder -->
+  <xacro:property name="link_radius" value="0.02"/>
+  <xacro:property name="link_length" value="3.0"/>
+  <xacro:property name="link_height_offset" value="0.5"/>
  <xacro:include filename="$(find ur_description)/urdf/inc/ur5_macro.xacro"/>
   <xacro:ur5_robot prefix="ur5_" />
-  <!-- Base cylinder -->
- <xacro:property name="link_radius" value="0.02"/>
-  <xacro:property name="link_length" value="3.0"/>
-  <xacro:property name="link_height_offset" value="0.5"/>
   <link name="base_link">
     <visual>
@@ -17,17 +17,4 @@
       </material>
     </visual>
-    <collision>
-      <origin xyz="0 0 ${link_height_offset}" rpy="0 0 0"/>
-      <geometry>
-        <cylinder radius="${link_radius}" length="${link_length}"/>
-      </geometry>
-    </collision>
-    <inertial>
-      <origin xyz="0 0 ${link_height_offset}" rpy="0 0 0"/>
-      <mass value="5.0"/>
-      <inertia ixx="0.1" ixy="0.0" ixz="0.0"
-               iyy="0.1" iyz="0.0"
-               izz="0.1"/>
-    </inertial>
   </link>
  <joint name="base_to_table" type="fixed">
@@ -37,33 +24,2 @@
   </joint>
 </robot>
-<?xml version="1.0"?>
-<robot xmlns:xacro="http://www.ros.org/wiki/xacro" name="my_robot">
-  <!-- Base cylinder -->
- <xacro:property name="link_radius" value="0.02"/>
-  <xacro:property name="link_length" value="3.0"/>
-  <xacro:property name="link_height_offset" value="0.5"/>
-  <link name="base_link">
-    <visual>
-      <origin xyz="0 0 ${link_height_offset}" rpy="0 0 0"/>
-      <geometry>
-        <cylinder radius="${link_radius}" length="${link_length}"/>
-      </geometry>
-      <material name="green">
-        <color rgba="1 0 0 1"/>
-      </material>
-    </visual>
-    <collision>
-      <origin xyz="0 0 ${link_height_offset}" rpy="0 0 0"/>
-      <geometry>
-        <cylinder radius="${link_radius}" length="${link_length}"/>
-      </geometry>
-    </collision>
-    <inertial>
-      <origin xyz="0 0 ${link_height_offset}" rpy="0 0 0"/>
-      <mass value="5.0"/>
-      <inertia ixx="0.1" ixy="0.0" ixz="0.0"
-               iyy="0.1" iyz="0.0"
-               izz="0.1"/>
-    </inertial>
-  </link>
-</robot>

Commit message: Update robot.xacro

File: my_robot_description/urdf/robot.xacro (robot description, xacro)
@@ -3,10 +3,9 @@
   <!-- Base cylinder -->
   <xacro:property name="link_radius" value="0.02"/>
-  <xacro:property name="link_length" value="3.0"/>
+  <xacro:property name="link_length" value="1.0"/>
   <xacro:property name="link_height_offset" value="0.5"/>
  <xacro:include filename="$(find ur_description)/urdf/inc/ur5_macro.xacro"/>
   <xacro:ur5_robot prefix="ur5_" />
 <xacro:include filename="$(find my_robot_description)/urdf/table.xacro"/>
-<xacro:wood_table name="bench" parent="base_link" x="1" y="0" z="0"/>
   <link name="base_link">
     <visual>
@@ -20,8 +19,13 @@
     </visual>
   </link>
- <joint name="base_to_table" type="fixed">
+  <joint name="table_joint" type="fixed">
     <parent link="base_link"/>
-    <child link="ur5_base_link"/>
+    <child link="table_link"/>
     <origin xyz="0 1 0.9" rpy="0 0 0"/>
   </joint>
+ <joint name="base_to_table" type="fixed">
+    <parent link="table_link"/>
+    <child link="ur5_base_link"/>
+    <origin xyz="0.2 0.2 0" rpy="0 0 0"/>
+  </joint>
 </robot>

Commit message: Update robot.xacro

File: my_robot_description/urdf/robot.xacro (robot description, xacro)
@@ -27,5 +27,5 @@
     <parent link="table_link"/>
     <child link="ur5_base_link"/>
-    <origin xyz="0.2 0.2 0" rpy="0 0 0"/>
+    <origin xyz="0.2 1.2 0" rpy="0 0 0"/>
   </joint>
 </robot>

Commit message: Update robot.xacro

File: my_robot_description/urdf/robot.xacro (robot description, xacro)
@@ -6,7 +6,7 @@
   <xacro:property name="link_height_offset" value="0.5"/>
  <xacro:include filename="$(find ur_description)/urdf/inc/ur5_macro.xacro"/>
-  <xacro:ur5_robot prefix="ur5_" />
+  <xacro:ur5_robot prefix="" />
 <xacro:include filename="$(find my_robot_description)/urdf/table.xacro"/>
-  <link name="base_link">
+  <link name="my_base_link">
     <visual>
       <origin xyz="0 0 ${link_height_offset}" rpy="0 0 0"/>
@@ -20,5 +20,5 @@
   </link>
   <joint name="table_joint" type="fixed">
-    <parent link="base_link"/>
+    <parent link="my_base_link"/>
     <child link="table_link"/>
     <origin xyz="0 1 0.9" rpy="0 0 0"/>
@@ -26,5 +26,5 @@
  <joint name="base_to_table" type="fixed">
     <parent link="table_link"/>
-    <child link="ur5_base_link"/>
+    <child link="base_link"/>
     <origin xyz="0.2 1.2 0" rpy="0 0 0"/>
   </joint>

Commit message: Update robot.xacro

File: my_robot_description/urdf/robot.xacro (robot description, xacro)
@@ -6,7 +6,7 @@
   <xacro:property name="link_height_offset" value="0.5"/>
  <xacro:include filename="$(find ur_description)/urdf/inc/ur5_macro.xacro"/>
-  <xacro:ur5_robot prefix="" />
+  <xacro:ur5_robot prefix="UR5_" />
 <xacro:include filename="$(find my_robot_description)/urdf/table.xacro"/>
-  <link name="my_base_link">
+  <link name="base_link">
     <visual>
       <origin xyz="0 0 ${link_height_offset}" rpy="0 0 0"/>
@@ -20,5 +20,5 @@
   </link>
   <joint name="table_joint" type="fixed">
-    <parent link="my_base_link"/>
+    <parent link="base_link"/>
     <child link="table_link"/>
     <origin xyz="0 1 0.9" rpy="0 0 0"/>
@@ -26,5 +26,5 @@
  <joint name="base_to_table" type="fixed">
     <parent link="table_link"/>
-    <child link="base_link"/>
+    <child link="UR5_base_link"/>
     <origin xyz="0.2 1.2 0" rpy="0 0 0"/>
   </joint>

Commit message: Update robot.xacro

File: my_robot_description/urdf/robot.xacro (robot description, xacro)
@@ -6,7 +6,7 @@
   <xacro:property name="link_height_offset" value="0.5"/>
  <xacro:include filename="$(find ur_description)/urdf/inc/ur5_macro.xacro"/>
-  <xacro:ur5_robot prefix="UR5_" />
+  <xacro:ur5_robot prefix="" />
 <xacro:include filename="$(find my_robot_description)/urdf/table.xacro"/>
-  <link name="base_link">
+  <link name="world">
     <visual>
       <origin xyz="0 0 ${link_height_offset}" rpy="0 0 0"/>
@@ -20,11 +20,11 @@
   </link>
   <joint name="table_joint" type="fixed">
-    <parent link="base_link"/>
+    <parent link="world"/>
     <child link="table_link"/>
     <origin xyz="0 1 0.9" rpy="0 0 0"/>
   </joint>
  <joint name="base_to_table" type="fixed">
-    <parent link="table_link"/>
-    <child link="UR5_base_link"/>
+    <parent link="world"/>
+    <child link="base_link"/>
     <origin xyz="0.2 1.2 0" rpy="0 0 0"/>
   </joint>

Commit message: Update robot.xacro

File: my_robot_description/urdf/robot.xacro (robot description, xacro)
@@ -8,5 +8,5 @@
   <xacro:ur5_robot prefix="" />
 <xacro:include filename="$(find my_robot_description)/urdf/table.xacro"/>
-  <link name="world">
+  <link name="test">
     <visual>
       <origin xyz="0 0 ${link_height_offset}" rpy="0 0 0"/>
@@ -20,11 +20,11 @@
   </link>
   <joint name="table_joint" type="fixed">
-    <parent link="world"/>
+    <parent link="base_link"/>
     <child link="table_link"/>
     <origin xyz="0 1 0.9" rpy="0 0 0"/>
   </joint>
  <joint name="base_to_table" type="fixed">
-    <parent link="world"/>
-    <child link="base_link"/>
+    <parent link="base_link"/>
+    <child link="test"/>
     <origin xyz="0.2 1.2 0" rpy="0 0 0"/>
   </joint>

Commit message: Update robot.xacro

File: my_robot_description/urdf/robot.xacro (robot description, xacro)
@@ -22,5 +22,5 @@
     <parent link="base_link"/>
     <child link="table_link"/>
-    <origin xyz="0 1 0.9" rpy="0 0 0"/>
+    <origin xyz="-0.9 -0.3 0" rpy="0 0 0"/>
   </joint>
  <joint name="base_to_table" type="fixed">
