Commit message: Update ur5_with_RGgripper.xacro

File: my_robot_description/urdf/ur5_with_RGgripper.xacro (robot description, xacro)
@@ -9,6 +9,11 @@
   <!-- GRIPPER ADDITION      -->
   <!-- ===================== -->
-  <xacro:include filename="$(find my_robot_description)/urdf/MyFingerGrip.xacro"/>
+ <xacro:include filename="$(find onrobot_rg_description)/urdf/onrobot_rg2_model_macro.xacro" />
+  <xacro:onrobot_rg2 prefix=""/>
   <!-- Attach gripper to tool0  this is default name of rosindustrial UR connection link -->
-  <xacro:MyFingerGrip parent="tool0"/>
+   <joint name="tool0_to_gripper" type="fixed">
+      <parent link="tool0"/>
+      <child link="onrobot_rg2_base_link"/>
+      <origin xyz="0 0 0.1" rpy="0 0 0"/>
+    </joint>
 </robot>

Commit message: Update ur5_with_RGgripper.xacro

File: my_robot_description/urdf/ur5_with_RGgripper.xacro (robot description, xacro)
@@ -1,4 +1,4 @@
 <?xml version="1.0"?>
-<robot xmlns:xacro="http://www.ros.org/wiki/xacro" name="ur5_with_gripper">
+<robot xmlns:xacro="http://www.ros.org/wiki/xacro" name="ur5_with_RGgripper">
   <!-- ===================== -->
   <!-- UR5 BASE ROBOT        -->
@@ -9,11 +9,11 @@
   <!-- GRIPPER ADDITION      -->
   <!-- ===================== -->
- <xacro:include filename="$(find onrobot_rg_description)/urdf/onrobot_rg2_model_macro.xacro" />
-  <xacro:onrobot_rg2 prefix=""/>
+ <xacro:include filename="$(find onrobot_rg_description)/urdf/onrobot_rg2.xacro" />
+  <xacro:onrobot_rg2 prefix="rg2_"/>
   <!-- Attach gripper to tool0  this is default name of rosindustrial UR connection link -->
-   <joint name="tool0_to_gripper" type="fixed">
-      <parent link="tool0"/>
-      <child link="onrobot_rg2_base_link"/>
-      <origin xyz="0 0 0.1" rpy="0 0 0"/>
-    </joint>
+<joint name="tool0_to_rg2" type="fixed">
+  <parent link="tool0"/>
+  <child link="rg2_onrobot_rg2_base_link"/>
+  <origin xyz="0 0 0" rpy="0 0 0"/>
+</joint>
 </robot>

Commit message: Update ur5_with_RGgripper.xacro

File: my_robot_description/urdf/ur5_with_RGgripper.xacro (robot description, xacro)
@@ -14,5 +14,5 @@
 <joint name="tool0_to_rg2" type="fixed">
   <parent link="tool0"/>
-  <child link="rg2_onrobot_rg2_base_link"/>
+  <child link="world"/>
   <origin xyz="0 0 0" rpy="0 0 0"/>
 </joint>

Commit message: Update ur5_with_RGgripper.xacro

File: my_robot_description/urdf/ur5_with_RGgripper.xacro (robot description, xacro)
@@ -9,11 +9,11 @@
   <!-- GRIPPER ADDITION      -->
   <!-- ===================== -->
- <xacro:include filename="$(find onrobot_rg_description)/urdf/onrobot_rg2.xacro" />
+  <xacro:include filename="$(find onrobot_rg_description)/urdf/onrobot_rg2_model_macro.xacro"/>
   <xacro:onrobot_rg2 prefix=""/>
-  <!-- Attach gripper to tool0  this is default name of rosindustrial UR connection link -->
-<joint name="tool0_to_rg2" type="fixed">
-  <parent link="tool0"/>
-  <child link="world"/>
-  <origin xyz="0 0 0" rpy="0 0 0"/>
-</joint>
+  <!-- attach gripper -->
+  <joint name="rg2_joint" type="fixed">
+    <parent link="tool0"/>
+    <child link="onrobot_rg2_base_link"/>
+    <origin xyz="0 0 0" rpy="0 0 0"/>
+  </joint>
 </robot>

Commit message: Update ur5_with_RGgripper.xacro

File: my_robot_description/urdf/ur5_with_RGgripper.xacro (robot description, xacro)
@@ -3,8 +3,7 @@
   <!-- ===================== -->
   <!-- UR5 BASE ROBOT        -->
-  <!-- =====================
+  <!-- ===================== -->
   <xacro:include filename="$(find ur_description)/urdf/inc/ur5_macro.xacro"/>
   <xacro:ur5_robot prefix="" />
--->
   <!-- ===================== -->
   <!-- GRIPPER ADDITION      -->
@@ -12,10 +11,9 @@
   <xacro:include filename="$(find onrobot_rg_description)/urdf/onrobot_rg2_model_macro.xacro"/>
   <xacro:onrobot_rg2 prefix=""/>
-  <!-- attach gripper
+  <!-- attach gripper -->
   <joint name="rg2_joint" type="fixed">
     <parent link="tool0"/>
-    <child link="onrobot_rg2_base_link"/>
+    <child link="world"/>
     <origin xyz="0 0 0" rpy="0 0 0"/>
   </joint>
- -->
 </robot>

Commit message: Update ur5_with_RGgripper.xacro

File: my_robot_description/urdf/ur5_with_RGgripper.xacro (robot description, xacro)
@@ -14,5 +14,5 @@
   <joint name="rg2_joint" type="fixed">
     <parent link="tool0"/>
-    <child link="world"/>
+    <child link="onrobot_rg2_base_link"/>
     <origin xyz="0 0 0" rpy="0 0 0"/>
   </joint>

Commit message: Update ur5_with_RGgripper.xacro

File: my_robot_description/urdf/ur5_with_RGgripper.xacro (robot description, xacro)
@@ -15,5 +15,5 @@
     <parent link="tool0"/>
     <child link="onrobot_rg2_base_link"/>
-    <origin xyz="0 0 0" rpy="0 0 0"/>
+    <origin xyz="0 0 0.2" rpy="0 0 0"/>
   </joint>
 </robot>
