Commit message: Update GoldbarrenGroup.xacro

File: my_robot_description/urdf/GoldbarrenGroup.xacro (robot description, xacro)
@@ -14,5 +14,5 @@
       <origin xyz="0 0 0" rpy="0 0 0" />
       <geometry>
-        <mesh scale="0.07" filename="package://GoldbarrenGroup_description/meshes/GoldbarrenPart.stl" />
+        <mesh scale="0.07" filename="package://my_robot_description/meshes/GoldbarrenPart.stl" />
       </geometry>
       <material name="Metall - 1600F (heiß)" />

Commit message: Update GoldbarrenGroup.xacro

File: my_robot_description/urdf/GoldbarrenGroup.xacro (robot description, xacro)
@@ -14,5 +14,5 @@
       <origin xyz="0 0 0" rpy="0 0 0" />
       <geometry>
-        <mesh scale="0.07" filename="package://my_robot_description/meshes/GoldbarrenPart.stl" />
+        <mesh filename="package://my_robot_description/meshes/GoldbarrenPart.stl" />
       </geometry>
       <material name="Metall - 1600F (heiß)" />
