Commit message: Update my_robot.srdf.xacro

File: my_robot_moveit_config/config/my_robot.srdf.xacro (robot description, xacro)
@@ -0,0 +1,56 @@
+<?xml version="1.0"?>
+<robot xmlns:xacro="http://www.ros.org/wiki/xacro" name="ur5_robot">
+  <!-- ========================= -->
+  <!-- Prefix argument -->
+  <!-- ========================= -->
+  <xacro:arg name="prefix" default=""/>
+  <!-- convenience macro -->
+  <xacro:property name="p" value="${prefix}"/>
+  <!-- ========================= -->
+  <!-- GROUPS -->
+  <!-- ========================= -->
+  <group name="manipulator">
+    <chain base_link="${p}base_link" tip_link="${p}tool0"/>
+  </group>
+  <!-- ========================= -->
+  <!-- GROUP STATES -->
+  <!-- ========================= -->
+  <group_state name="home" group="manipulator">
+    <joint name="${p}elbow_joint" value="0" />
+    <joint name="${p}shoulder_lift_joint" value="0" />
+    <joint name="${p}shoulder_pan_joint" value="0" />
+    <joint name="${p}wrist_1_joint" value="0" />
+    <joint name="${p}wrist_2_joint" value="0" />
+    <joint name="${p}wrist_3_joint" value="0" />
+  </group_state>
+  <group_state name="up" group="manipulator">
+    <joint name="${p}elbow_joint" value="0" />
+    <joint name="${p}shoulder_lift_joint" value="-1.5707" />
+    <joint name="${p}shoulder_pan_joint" value="0" />
+    <joint name="${p}wrist_1_joint" value="-1.5707" />
+    <joint name="${p}wrist_2_joint" value="0" />
+    <joint name="${p}wrist_3_joint" value="0" />
+  </group_state>
+  <!-- ========================= -->
+  <!-- VIRTUAL JOINT -->
+  <!-- ========================= -->
+  <virtual_joint name="fixed_base"
+                 type="fixed"
+                 parent_frame="world"
+                 child_link="${p}base_link" />
+  <!-- ========================= -->
+  <!-- DISABLE COLLISIONS -->
+  <!-- (links usually do NOT change with prefix) -->
+  <!-- ========================= -->
+  <disable_collisions link1="base_link_inertia" link2="shoulder_link" reason="Adjacent" />
+  <disable_collisions link1="base_link_inertia" link2="upper_arm_link" reason="Never" />
+  <disable_collisions link1="base_link_inertia" link2="wrist_1_link" reason="Never" />
+  <disable_collisions link1="forearm_link" link2="upper_arm_link" reason="Adjacent" />
+  <disable_collisions link1="forearm_link" link2="wrist_1_link" reason="Adjacent" />
+  <disable_collisions link1="shoulder_link" link2="upper_arm_link" reason="Adjacent" />
+  <disable_collisions link1="shoulder_link" link2="wrist_1_link" reason="Never" />
+  <disable_collisions link1="shoulder_link" link2="wrist_2_link" reason="Never" />
+  <disable_collisions link1="wrist_1_link" link2="wrist_2_link" reason="Adjacent" />
+  <disable_collisions link1="wrist_1_link" link2="wrist_3_link" reason="Never" />
+  <disable_collisions link1="wrist_2_link" link2="wrist_3_link" reason="Adjacent" />
+</robot>
